File: KNEE CONTROLLER PCBA.kicad_pcb (KiCad board)
At the start: 2 copper layers, 60 x 120 mm, 166 parts, among them J1 VIN_CONN, J10 SW2_CONN, J11 CAN_CONN, J12 I2C_CONN, J13 SW3_CONN, J14 ST-LINK_CONN, J15 TEMP_CONN, J16 AUX_ADC_CONN, J17 TAG_CONN, J18 SW4_CONN, J2 MOT_CONN, J3 DRV_DIAG, J4 DRV_SKT_LEFT, J5 DRV_SKT_RIGHT, J6 USB_CONN, J7 ENC_CONN, J8 SW1_CONN, J9 UART_CONN, Q1 UTT18P10L-TN3-R, Q2 NCE0106R, SW1 SW_RESET, SW2 SW_CAN_TERM, SW3 SW_USER, U1 LMR36510ADDAR, U3 AP7362-33SP-13, U4 TLV6700QDDCRQ1, U5 INA238AIDGSR, U6 STM32L476RGT6, U7 TLV4041R5DBVR, U8 TJA1051T-3-1J-TD, U9 USBLC6-2SC6, Y1 ECS-80-8-30-JGN-TR, Y2 ECS-.327-6-34R-TR

Commit message: chore(template): update project files
Parts:
- added ID2: BOARD_IDENTIFICATION_MARKER, RD-Symbols-Silkscreen:BOARD_IDENTIFICATION, F.Cu at (241.3, 166.2)
- J16: value AUX_ADC_CONN -> ADC_CONN
- moved ID1 2.69 mm to (236.8, 174.7)
Routing:
- net GND: vias 389 -> 377

Commit message: chore(pcb): update project files
Parts:
- J1: footprint Connector_Molex:Molex_Micro-Fit_3.0_43650-0215_1x02_P3.00mm_Vertical -> Connector_Molex_Addendum:Molex_Micro-Fit_3.0_43650-0215_1x02_P3.00mm_Vertical
- J2: footprint Connector_Molex:Molex_Micro-Fit_3.0_43650-0415_1x04_P3.00mm_Vertical -> Connector_Molex_Addendum:Molex_Micro-Fit_3.0_43650-0415_1x04_P3.00mm_Vertical
- Q1: value UTT18P10L-TN3-R -> CRTD700P10L

Commit message: chore(pcb): update project files
Parts:
- C24, C27: value 10p -> 30p
- C28, C29, C30, C36: footprint Capacitor_SMD:C_0603_1608Metric -> Capacitor_SMD:C_0805_2012Metric
- C33, C34: value 10p -> 15p
- FH1: value XF-508P-B-B -> VIN_FH
- U8: value TJA1051T-3-1J-TD -> TJA1051T/3
- Y1: value ECS-80-8-30-JGN-TR -> X50328MSB2GI
- Y2: value ECS-.327-6-34R-TR -> Q13FC13500004
- moved C30 0.64 mm to (215.9, 125.9)
- moved C28 0.32 mm to (215.8, 138.0)
- turned C27 to 180 degrees
- turned C34 to 180 degrees
Connections:
- C27 pad 1: /PROJECT/XTAL -> GND
- C27 pad 2: GND -> /PROJECT/XTAL
- C34 pad 1: /PROJECT/OSC32_OUT -> GND
- C34 pad 2: GND -> /PROJECT/OSC32_OUT
Routing:
- net VDD: track 36.4 -> 1.92 mm
- net /PROJECT/BRAKE_GATE: track 6.09 -> 0.03 mm
- net /PROJECT/VM_OV_SENSE: track 4.89 -> 0.07 mm
- net /PROJECT/VM_UV_SENSE: track 4.86 -> 0.33 mm
- net +3V3: track 361.0 -> 357.4 mm
- net /PROJECT/BRAKE_SENSE: track 3.31 -> 0.00 mm
- net GND: track 80.8 -> 77.9 mm, vias 377 -> 374
- net /PROJECT/~{VM_UV}: track 49.7 -> 48.3 mm
- net /PROJECT/~{VM_OV}: track 51.8 -> 50.4 mm
- added copper zone on F.Cu, net /PROJECT/BRAKE_GATE
- added copper zone on F.Cu, net /PROJECT/BRAKE_SENSE
- added copper zone on F.Cu, net /PROJECT/VM_OV_SENSE
- added copper zone on F.Cu, net /PROJECT/VM_UV_SENSE
- added copper zone on F.Cu, net /PROJECT/~{VM_OV}
- added copper zone on F.Cu, net /PROJECT/~{VM_UV}
Other:
- board text added: "36V NOM 42V MAX 5A FUSE"
- board text added: "A1"
- board text added: "A2"
- board text added: "B1"
- board text added: "B2"
- board text added: "INT"
- board text added: "USB"

Commit message: chore(pcb): update project files
Routing:
- net +3V3: track 357.4 -> 340.3 mm
Other:
- board text added: "+3V3"
- board text added: "+5V"
- board text added: "+VUSB"
- board text added: "CLK"
- board text added: "GND"
