File: KNEE CONTROLLER PCBA.kicad_pcb (KiCad board)
At the start: 2 copper layers, 60 x 120 mm, 167 parts, among them J1 VIN_CONN, J10 SW2_CONN, J11 CAN_CONN, J12 I2C_CONN, J13 SW3_CONN, J14 ST-LINK_CONN, J15 TEMP_CONN, J16 ADC_CONN, J17 TAG_CONN, J18 SW4_CONN, J2 MOT_CONN, J3 DRV_DIAG, J4 DRV_SKT_LEFT, J5 DRV_SKT_RIGHT, J6 USB_CONN, J7 ENC_CONN, J8 SW1_CONN, J9 UART_CONN, Q1 CRTD700P10L, Q2 NCE0106R, SW1 SW_RESET, SW2 SW_CAN_TERM, SW3 SW_USER, U1 LMR36510ADDAR, U3 AP7362-33SP-13, U4 TLV6700QDDCRQ1, U5 INA238AIDGSR, U6 STM32L476RGT6, U7 TLV4041R5DBVR, U8 TJA1051T/3, U9 USBLC6-2SC6, Y1 X50328MSB2GI, Y2 Q13FC13500004

Commit message: chore(pcb): update project files
Parts:
- added C47: 10n, Capacitor_SMD:C_0603_1608Metric, F.Cu at (208.3, 79.0)
- added R55: 1k, Resistor_SMD:R_0603_1608Metric, F.Cu at (209.1, 74.8)
- added TP10: TEMP_ADC, RD-Testpoints:TestPoint_Pad_D0.4mm, F.Cu at (210.7, 90.1)
- added TP13: GND, RD-Testpoints:TestPoint_Pad_1.0x1.0mm, F.Cu at (225.9, 109.1)
- added TP14: AUX_ADC, RD-Testpoints:TestPoint_Pad_D0.4mm, F.Cu at (209.4, 90.1)
- added TP6: ~{VM_UV}, RD-Testpoints:TestPoint_Pad_D0.4mm, F.Cu at (211.6, 118.0)
- added TP7: ~{VM_OV}, RD-Testpoints:TestPoint_Pad_D0.4mm, F.Cu at (212.3, 114.8)
- added TP8: ~{VM_ALERT}, RD-Testpoints:TestPoint_Pad_D0.4mm, F.Cu at (212.9, 111.7)
- renumbered R55 to R56, TP7 to TP11, TP8 to TP12, TP6 to TP9
Connections:
- J16 pad 3: /PROJECT/AUX_ADC -> /PROJECT/AUX_ADC_CONN
Routing:
- net /PROJECT/AUX_ADC: track 23.7 -> 18.1 mm
- net /PROJECT/AUX_ADC_CONN: track 0.00 -> 4.72 mm
- net /PROJECT/DRV_STEP: track 13.4 -> 12.6 mm
- net GND: vias 374 -> 375

Commit message: chore(pcb): update project files
Parts:
- removed the C44 at (213.5, 75.0)
- removed C47: 10n, Capacitor_SMD:C_0603_1608Metric
- removed U9: USBLC6-2SC6, Package_TO_SOT_SMD:SOT-23-6
- added C42: 10n, Capacitor_SMD:C_0603_1608Metric, F.Cu at (208.3, 79.0)
- added U7: USBLC6-2SC6, Package_TO_SOT_SMD:SOT-23-6, F.Cu at (230.0, 143.4)
- C41: renamed from C4; value 2.2u -> 1u; footprint Capacitor_SMD:C_1206_3216Metric -> Capacitor_SMD:C_0805_2012Metric
- R51: renamed from R52; value 1k -> 100
- TP2: renamed from TP8; value ~{VM_ALERT} -> VM_ALERT_N
- TP5: renamed from TP6; value ~{VM_UV} -> VM_UV_N
- TP6: renamed from TP7; value ~{VM_OV} -> VM_OV_N
- moved C41 92.2 mm to (213.4, 75.0), turned to -90 degrees
- moved C8 2.54 mm to (220.5, 166.9)
- turned R51 to 180 degrees
- renumbered C26 to C1, C15 to C10, C28 to C11, C1 to C12, C6 to C13, C7 to C14, C29 to C15, C8 to C16, C30 to C17, C36 to C18, C38 to C19, C35 to C2, C37 to C20, C39 to C21, C40 to C22, C45 to C23, C27 to C25, C33 to C26, C34 to C27, C9 to C28, C17 to C29, C2 to C3, C10 to C30, C11 to C31, C12 to C32, C18 to C33, C19 to C34, C13 to C35, C20 to C36, C14 to C37, C21 to C38, C22 to C39, C31 to C4, C23 to C40, C41 to C43, C42 to C44, C43 to C45, C32 to C5, C25 to C6, C16 to C7, C3 to C8, C5 to C9, D5 to D4, D4 to D5, J16 to J10, J7 to J11, J9 to J12, J11 to J13, J12 to J14, J8 to J15, J10 to J16, J13 to J17, J6 to J2, J14 to J3, J17 to J4, J15 to J5, J3 to J6, J4 to J7, J5 to J8, J2 to J9, JP4 to JP1, JP3 to JP2, JP2 to JP3, JP1 to JP4, R27 to R1, R28 to R10, R30 to R11, R25 to R12, R9 to R13, R26 to R14, R1 to R15, R10 to R16, R13 to R17, R14 to R18, R2 to R19, R29 to R2, R7 to R20, R3 to R21, R17 to R22, R36 to R23, R39 to R24, R40 to R25, R37 to R26, R38 to R27, R46 to R28, R51 to R29, R19 to R3, R43 to R30, R47 to R31, R50 to R32, R48 to R33, R35 to R34, R45 to R35, R53 to R36, R56 to R37, R15 to R38, R31 to R39, R8 to R4, R32 to R40, R11 to R41, R33 to R42, R16 to R43, R22 to R44, R34 to R45, R23 to R46, R24 to R47, R4 to R48, R5 to R49, R6 to R5, R49 to R50, R55 to R52, R41 to R53, R42 to R54, R44 to R55, R54 to R56, R21 to R6, R12 to R7, R18 to R8, R20 to R9, SW2 to SW1, SW3 to SW2, SW1 to SW3, TP11 to TP10, TP12 to TP11, TP13 to TP12, TP10 to TP13, TP2 to TP3, TP3 to TP4, TP4 to TP7, TP5 to TP8, U5 to U1, U7 to U2, U4 to U3, U1 to U4, U3 to U5, U8 to U6, U6 to U8
Connections:
- net /PROJECT/A1 renamed /SYSTEM OVERVIEW/MOTOR CONTROL AND IO/A1
- net /PROJECT/A2 renamed /SYSTEM OVERVIEW/MOTOR CONTROL AND IO/A2
- net /PROJECT/AUX_ADC renamed /SYSTEM OVERVIEW/MICROCONTROLLER/AUX_ADC
- net /PROJECT/AUX_ADC_CONN renamed /SYSTEM OVERVIEW/MOTOR CONTROL AND IO/AUX_ADC_CONN
- net /PROJECT/AUX_UART_RX renamed /SYSTEM OVERVIEW/MICROCONTROLLER/AUX_UART_RX
- net /PROJECT/AUX_UART_TX renamed /SYSTEM OVERVIEW/MICROCONTROLLER/AUX_UART_TX
- net /PROJECT/B1 renamed /SYSTEM OVERVIEW/MOTOR CONTROL AND IO/B1
- net /PROJECT/B2 renamed /SYSTEM OVERVIEW/MOTOR CONTROL AND IO/B2
- net /PROJECT/BOOT renamed /SYSTEM OVERVIEW/POWER MANAGEMENT/BOOT
- net /PROJECT/BOOT0 renamed /SYSTEM OVERVIEW/MICROCONTROLLER/BOOT0
- net /PROJECT/BRAKE_ACTIVE renamed /SYSTEM OVERVIEW/MICROCONTROLLER/BRAKE_ACTIVE
- net /PROJECT/BRAKE_CMD renamed /SYSTEM OVERVIEW/POWER MANAGEMENT/BRAKE_CMD
- net /PROJECT/BRAKE_DRAIN renamed /SYSTEM OVERVIEW/POWER MANAGEMENT/BRAKE_DRAIN
- net /PROJECT/BRAKE_GATE renamed /SYSTEM OVERVIEW/POWER MANAGEMENT/BRAKE_GATE
- net /PROJECT/BRAKE_SENSE renamed /SYSTEM OVERVIEW/POWER MANAGEMENT/BRAKE_SENSE
- net /PROJECT/CAN_120R_SW renamed /SYSTEM OVERVIEW/MICROCONTROLLER/CAN_120R_SW
- net /PROJECT/CAN_H renamed /SYSTEM OVERVIEW/MICROCONTROLLER/CAN_H
- net /PROJECT/CAN_H_INT renamed /SYSTEM OVERVIEW/MICROCONTROLLER/CAN_H_INT
- net /PROJECT/CAN_L renamed /SYSTEM OVERVIEW/MICROCONTROLLER/CAN_L
- net /PROJECT/CAN_L_INT renamed /SYSTEM OVERVIEW/MICROCONTROLLER/CAN_L_INT
- net /PROJECT/CAN_RX renamed /SYSTEM OVERVIEW/MICROCONTROLLER/CAN_RX
- net /PROJECT/CAN_S renamed /SYSTEM OVERVIEW/MICROCONTROLLER/CAN_S
- net /PROJECT/CAN_TX renamed /SYSTEM OVERVIEW/MICROCONTROLLER/CAN_TX
- net /PROJECT/CC1 renamed /SYSTEM OVERVIEW/MICROCONTROLLER/CC1
- net /PROJECT/CC2 renamed /SYSTEM OVERVIEW/MICROCONTROLLER/CC2
- net /PROJECT/CONF_PULLUP renamed /SYSTEM OVERVIEW/MOTOR CONTROL AND IO/CONF_PULLUP
- net /PROJECT/DBG_SWCLK renamed /SYSTEM OVERVIEW/MICROCONTROLLER/DBG_SWCLK
- net /PROJECT/DBG_SWCLK_CONN renamed /SYSTEM OVERVIEW/MICROCONTROLLER/DBG_SWCLK_CONN
- net /PROJECT/DBG_SWDIO renamed /SYSTEM OVERVIEW/MICROCONTROLLER/DBG_SWDIO
- net /PROJECT/DBG_SWDIO_CONN renamed /SYSTEM OVERVIEW/MICROCONTROLLER/DBG_SWDIO_CONN
- net /PROJECT/DBG_SWO renamed /SYSTEM OVERVIEW/MICROCONTROLLER/DBG_SWO
- net /PROJECT/DBG_SWO_CONN renamed /SYSTEM OVERVIEW/MICROCONTROLLER/DBG_SWO_CONN
- net /PROJECT/DBG_UART_RX renamed /SYSTEM OVERVIEW/MICROCONTROLLER/DBG_UART_RX
- net /PROJECT/DBG_UART_RX_CONN renamed /SYSTEM OVERVIEW/MICROCONTROLLER/DBG_UART_RX_CONN
- net /PROJECT/DBG_UART_TX renamed /SYSTEM OVERVIEW/MICROCONTROLLER/DBG_UART_TX
- net /PROJECT/DBG_UART_TX_CONN renamed /SYSTEM OVERVIEW/MICROCONTROLLER/DBG_UART_TX_CONN
- net /PROJECT/DRV_CLK renamed /SYSTEM OVERVIEW/MOTOR CONTROL AND IO/DRV_CLK
- net /PROJECT/DRV_CSN renamed /SYSTEM OVERVIEW/MOTOR CONTROL AND IO/DRV_CS
- net /PROJECT/DRV_DIAG0 renamed /SYSTEM OVERVIEW/MOTOR CONTROL AND IO/DRV_DIAG0
- net /PROJECT/DRV_DIAG1 renamed /SYSTEM OVERVIEW/MOTOR CONTROL AND IO/DRV_DIAG1
- net /PROJECT/DRV_DIR renamed /SYSTEM OVERVIEW/MOTOR CONTROL AND IO/DRV_DIR
- net /PROJECT/DRV_SCK renamed /SYSTEM OVERVIEW/MOTOR CONTROL AND IO/DRV_SCK
- net /PROJECT/DRV_SDI renamed /SYSTEM OVERVIEW/MOTOR CONTROL AND IO/DRV_MOSI
- net /PROJECT/DRV_SDO renamed /SYSTEM OVERVIEW/MOTOR CONTROL AND IO/DRV_MISO
- net /PROJECT/DRV_STEP renamed /SYSTEM OVERVIEW/MOTOR CONTROL AND IO/DRV_STEP
- net /PROJECT/ENC_AUX_SCK renamed /SYSTEM OVERVIEW/MICROCONTROLLER/ENC_AUX_SCK
- net /PROJECT/ENC_A_MISO renamed /SYSTEM OVERVIEW/MICROCONTROLLER/ENC_A_MISO
- net /PROJECT/ENC_B_MOSI renamed /SYSTEM OVERVIEW/MICROCONTROLLER/ENC_B_MOSI
- net /PROJECT/ENC_Z_CS renamed /SYSTEM OVERVIEW/MICROCONTROLLER/ENC_Z_CS
- net /PROJECT/FB renamed /SYSTEM OVERVIEW/POWER MANAGEMENT/FB
- net /PROJECT/I2C1_SCL renamed /SYSTEM OVERVIEW/MICROCONTROLLER/I2C1_SCL
- net /PROJECT/I2C1_SDA renamed /SYSTEM OVERVIEW/MICROCONTROLLER/I2C1_SDA
- net /PROJECT/I2C2_SCL renamed /SYSTEM OVERVIEW/MICROCONTROLLER/I2C2_SCL
- net /PROJECT/I2C2_SDA renamed /SYSTEM OVERVIEW/MICROCONTROLLER/I2C2_SDA
- net /PROJECT/INA_INN renamed /SYSTEM OVERVIEW/POWER MANAGEMENT/INA_INN
- net /PROJECT/INA_INP renamed /SYSTEM OVERVIEW/POWER MANAGEMENT/INA_INP
- net /PROJECT/LED_GRN renamed /SYSTEM OVERVIEW/MICROCONTROLLER/LED_YEL
- net /PROJECT/LED_RED renamed /SYSTEM OVERVIEW/MICROCONTROLLER/LED_RED
- net /PROJECT/OSC32_IN renamed /SYSTEM OVERVIEW/MICROCONTROLLER/OSC32_IN
- net /PROJECT/OSC32_OUT renamed /SYSTEM OVERVIEW/MICROCONTROLLER/OSC32_OUT
- net /PROJECT/OSC_IN renamed /SYSTEM OVERVIEW/MICROCONTROLLER/OSC_IN
- net /PROJECT/OSC_OUT renamed /SYSTEM OVERVIEW/MICROCONTROLLER/OSC_OUT
- net /PROJECT/PWR_3V3_OK renamed /SYSTEM OVERVIEW/POWER MANAGEMENT/PWR_3V3_OK
- net /PROJECT/PWR_5V_OK renamed /SYSTEM OVERVIEW/POWER MANAGEMENT/PWR_5V_OK
- net /PROJECT/RPP_GATE renamed /SYSTEM OVERVIEW/POWER MANAGEMENT/RPP_GATE
- net /PROJECT/SW renamed /SYSTEM OVERVIEW/POWER MANAGEMENT/SW
- net /PROJECT/SW1_SIG renamed /SYSTEM OVERVIEW/MICROCONTROLLER/SW1_SIG
- net /PROJECT/SW1_SIG_MCU renamed /SYSTEM OVERVIEW/MICROCONTROLLER/SW1_SIG_MCU
- net /PROJECT/SW2_SIG renamed /SYSTEM OVERVIEW/MICROCONTROLLER/SW2_SIG
- net /PROJECT/SW2_SIG_MCU renamed /SYSTEM OVERVIEW/MICROCONTROLLER/SW2_SIG_MCU
- net /PROJECT/SW3_SIG renamed /SYSTEM OVERVIEW/MICROCONTROLLER/SW3_SIG
- net /PROJECT/SW3_SIG_MCU renamed /SYSTEM OVERVIEW/MICROCONTROLLER/SW3_SIG_MCU
- net /PROJECT/SW4_SIG renamed /SYSTEM OVERVIEW/MICROCONTROLLER/SW4_SIG
- net /PROJECT/SW4_SIG_MCU renamed /SYSTEM OVERVIEW/MICROCONTROLLER/SW4_SIG_MCU
- net /PROJECT/USB_CONN+ renamed /SYSTEM OVERVIEW/MICROCONTROLLER/USB_CONN+
- net /PROJECT/USB_CONN- renamed /SYSTEM OVERVIEW/MICROCONTROLLER/USB_CONN-
- net /PROJECT/VCC renamed /SYSTEM OVERVIEW/POWER MANAGEMENT/VCC
- net /PROJECT/VIN_SEL renamed /SYSTEM OVERVIEW/POWER MANAGEMENT/VIN_SEL
- net /PROJECT/VM_OV_SENSE renamed /SYSTEM OVERVIEW/POWER MANAGEMENT/VM_OV_SENSE
- net /PROJECT/VM_UV_SENSE renamed /SYSTEM OVERVIEW/POWER MANAGEMENT/VM_UV_SENSE
- net /PROJECT/XTAL renamed /SYSTEM OVERVIEW/MICROCONTROLLER/XTAL
- net /PROJECT/~{BTN} renamed /SYSTEM OVERVIEW/MICROCONTROLLER/BTN_N
- net /PROJECT/~{DBG_RST_CONN} renamed /SYSTEM OVERVIEW/MICROCONTROLLER/DBG_RST_CONN_N
- net /PROJECT/~{DBG_RST} renamed /SYSTEM OVERVIEW/MICROCONTROLLER/DBG_RST_N
- net /PROJECT/~{DRV_EN} renamed /SYSTEM OVERVIEW/MOTOR CONTROL AND IO/DRV_EN_N
- net /PROJECT/~{VM_ALERT} renamed /SYSTEM OVERVIEW/MICROCONTROLLER/VM_ALERT_N
- net /PROJECT/~{VM_OV} renamed /SYSTEM OVERVIEW/MICROCONTROLLER/VM_OV_N
- net /PROJECT/~{VM_UV} renamed /SYSTEM OVERVIEW/MICROCONTROLLER/VM_UV_N
- C41 pad 1: VIN_PROT -> GND
- C41 pad 2: GND -> /SYSTEM OVERVIEW/MICROCONTROLLER/TEMP_ADC
- J5 pad 2: /PROJECT/TEMP_NTC -> /SYSTEM OVERVIEW/MOTOR CONTROL AND IO/TEMP_NTC
- R50 pad 1: /PROJECT/TEMP_NTC -> /SYSTEM OVERVIEW/MOTOR CONTROL AND IO/TEMP_NTC
- R51 pad 1: /PROJECT/TEMP_ADC -> /SYSTEM OVERVIEW/MOTOR CONTROL AND IO/TEMP_NTC
- R51 pad 2: /PROJECT/TEMP_NTC -> /SYSTEM OVERVIEW/MICROCONTROLLER/TEMP_ADC
- TP13 pad 1: /PROJECT/TEMP_ADC -> /SYSTEM OVERVIEW/MICROCONTROLLER/TEMP_ADC
- U8 pad 10: /PROJECT/TEMP_ADC -> /SYSTEM OVERVIEW/MICROCONTROLLER/TEMP_ADC
- U8 pad 44: /PROJECT/USB_MCU- -> /SYSTEM OVERVIEW/MICROCONTROLLER/USB_MCU-
- U8 pad 45: /PROJECT/USB_MCU+ -> /SYSTEM OVERVIEW/MICROCONTROLLER/USB_MCU+
Routing:
- net /SYSTEM OVERVIEW/MICROCONTROLLER/USB_MCU-: track 0.00 -> 48.1 mm
- net /PROJECT/USB_MCU-: track 48.1 -> 0.00 mm
- net /SYSTEM OVERVIEW/MICROCONTROLLER/USB_MCU+: track 0.00 -> 48.1 mm
- net /PROJECT/USB_MCU+: track 48.1 -> 0.00 mm
- net /SYSTEM OVERVIEW/MICROCONTROLLER/TEMP_ADC: track 0.00 -> 22.3 mm
- net /PROJECT/TEMP_ADC: track 22.1 -> 0.00 mm
- net /SYSTEM OVERVIEW/MOTOR CONTROL AND IO/TEMP_NTC: track 0.00 -> 8.22 mm
- net /PROJECT/TEMP_NTC: track 8.22 -> 0.00 mm
- net /SYSTEM OVERVIEW/POWER MANAGEMENT/RPP_GATE: track 6.72 -> 0.00 mm
- net GND: track 77.9 -> 78.8 mm, vias 375 -> 376
- net +5V: track 284.5 -> 285.2 mm
- added copper zone on F.Cu, net /SYSTEM OVERVIEW/POWER MANAGEMENT/RPP_GATE
