File: KNEE CONTROLLER PCBA.kicad_pcb (KiCad board)
At the start: 2 copper layers, 60 x 120 mm, 174 parts, among them J1 VIN_CONN, J10 ADC_CONN, J11 ENC_CONN, J12 UART_CONN, J13 CAN_CONN, J14 I2C_CONN, J15 SW1_CONN, J16 SW2_CONN, J17 SW3_CONN, J18 SW4_CONN, J2 USB_CONN, J3 ST-LINK_CONN, J4 TAG_CONN, J5 TEMP_CONN, J6 DRV_DIAG, J7 DRV_SKT_LEFT, J8 DRV_SKT_RIGHT, J9 MOT_CONN, Q1 CRTD700P10L, Q2 NCE0106R, SW1 SW_CAN_TERM, SW2 SW_USER, SW3 SW_RESET, U1 INA238AIDGSR, U2 TLV4041R5DBVR, U3 TLV6700QDDCRQ1, U4 LMR36510ADDAR, U5 AP7362-33SP-13, U6 TJA1051T/3, U7 USBLC6-2SC6, U8 STM32L476RGT6, Y1 X50328MSB2GI, Y2 Q13FC13500004

Commit message: chore(pcb): update project files
Parts:
- added TP12: CAN_H, RD-Testpoints:TestPoint_Pad_D0.4mm, F.Cu at (221.4, 74.2)
- added TP13: CAN_L, RD-Testpoints:TestPoint_Pad_D0.4mm, F.Cu at (235.1, 74.2)
- added TP15: I2C2_SDA, RD-Testpoints:TestPoint_Pad_D0.4mm, F.Cu at (200.2, 102.6)
- added TP16: I2C2_SCL, RD-Testpoints:TestPoint_Pad_D0.4mm, F.Cu at (196.9, 104.0)
- added TP17: I2C1_SDA, RD-Testpoints:TestPoint_Pad_D0.4mm, F.Cu at (220.5, 97.0)
- added TP18: I2C1_SCL, RD-Testpoints:TestPoint_Pad_D0.4mm, F.Cu at (224.6, 97.6)
- added TP20: GND, RD-Testpoints:TestPoint_Pad_1.0x1.0mm, F.Cu at (202.4, 76.1)
- added TP7: SW, RD-Testpoints:TestPoint_Pad_D0.4mm, F.Cu at (229.4, 180.6)
- added TP8: VIN_SEL, RD-Testpoints:TestPoint_Pad_D0.4mm, F.Cu at (223.1, 153.6)
- added TP9: FB, RD-Testpoints:TestPoint_Pad_D0.4mm, F.Cu at (214.2, 178.0)
- renumbered TP7 to TP10, TP8 to TP11, TP9 to TP14, TP10 to TP19, TP11 to TP21, TP12 to TP22, TP13 to TP23, TP14 to TP24
Routing:
- net /SYSTEM OVERVIEW/MICROCONTROLLER/CAN_H: track 10.1 -> 13.0 mm
- net /SYSTEM OVERVIEW/MICROCONTROLLER/CAN_L: track 16.7 -> 19.2 mm
- net GND: vias 376 -> 453

Commit message: docs(docs): update project files
Parts:
- added TP19: CAN_RX, 0_RD_Testpoint:TestPoint_Pad_D0.4mm, F.Cu at (229.0, 87.1)
- added TP2: BRAKE_SENSE, 0_RD_Testpoint:TestPoint_Pad_D0.4mm, F.Cu at (190.9, 134.9)
- added TP20: CAN _TX, 0_RD_Testpoint:TestPoint_Pad_D0.4mm, F.Cu at (227.4, 87.8)
- added TP21: CAN_S, 0_RD_Testpoint:TestPoint_Pad_D0.4mm, F.Cu at (224.7, 87.1)
- added TP26: DBG_RST_N, 0_RD_Testpoint:TestPoint_Pad_D0.4mm, F.Cu at (222.4, 110.0)
- added TP31: DRV_MISO, 0_RD_Testpoint:TestPoint_Pad_D0.4mm, F.Cu at (205.7, 109.2)
- added TP32: DRV_MOSI, 0_RD_Testpoint:TestPoint_Pad_D0.4mm, F.Cu at (207.4, 108.2)
- added TP33: DRV_SCK, 0_RD_Testpoint:TestPoint_Pad_D0.4mm, F.Cu at (205.9, 108.2)
- added TP34: DRV_CS, 0_RD_Testpoint:TestPoint_Pad_D0.4mm, F.Cu at (204.1, 109.2)
- added TP35: DRV_DIR, 0_RD_Testpoint:TestPoint_Pad_D0.4mm, F.Cu at (209.5, 108.2)
- added TP36: DRV_EN_N, 0_RD_Testpoint:TestPoint_Pad_D0.4mm, F.Cu at (210.7, 109.2)
- added TP37: STEP_DIR, 0_RD_Testpoint:TestPoint_Pad_D0.4mm, F.Cu at (207.7, 109.2)
- added TP39: ENC_AUX_SCK, 0_RD_Testpoint:TestPoint_Pad_D0.4mm, F.Cu at (198.0, 92.2)
- added TP4: RPP_GATE, 0_RD_Testpoint:TestPoint_Pad_D0.4mm, F.Cu at (195.5, 168.4)
- added TP40: ENC_A_MISO, 0_RD_Testpoint:TestPoint_Pad_D0.4mm, F.Cu at (196.8, 93.5)
- added TP41: ENC_B_MOSI, 0_RD_Testpoint:TestPoint_Pad_D0.4mm, F.Cu at (195.5, 94.8)
- added TP42: ENC_Z_CS, 0_RD_Testpoint:TestPoint_Pad_D0.4mm, F.Cu at (199.3, 91.0)
- added TP5: BRAKE_CMD, 0_RD_Testpoint:TestPoint_Pad_D0.4mm, F.Cu at (199.1, 108.0)
- added TP6: BRAKE_GATE, 0_RD_Testpoint:TestPoint_Pad_D0.4mm, F.Cu at (189.9, 141.5)
- C1, C12, C16, C19, C2, C20, C21, C22, C23, C24, C25, C29, C30, C31, C32, C33, C34, C35, C38, C4, C42, C43, C44, C45, C46, C5, C6, C7: footprint Capacitor_SMD:C_0603_1608Metric -> 0_RD_Capacitor_SMD:C_0603_1608_DensityHigh
- C10, C11, C15, C17, C18, C36, C37, C41: footprint Capacitor_SMD:C_0805_2012Metric -> 0_RD_Capacitor_SMD:C_0805_2012_DensityHigh
- C13, C14, C28, C39, C8, C9: footprint Capacitor_SMD:C_1206_3216Metric -> 0_RD_Capacitor_SMD:C_1206_3216_DensityHigh
- C26, C27: footprint Capacitor_SMD:C_0402_1005Metric -> 0_RD_Capacitor_SMD:C_0402_1005_DensityHigh
- D1: footprint Diode_SMD:D_SOD-323_HandSoldering -> 0_RD_Diode_SMD:D_SOD-323
- D2, D3, D6, D7: footprint LED_SMD:LED_0805_2012Metric -> 0_RD_LED_SMD:LED_0805_2012_DensityHigh
- D5: value TVS -> SMBJ5.0A-TR; footprint Diode_SMD:D_SMB -> 0_RD_Diode_SMD:D_SMB
- FB1: footprint Inductor_SMD:L_0603_1608Metric -> 0_RD_Resistor_SMD:R_0603_1608_DensityHigh
- FID1, FID2, FID3: footprint Fiducial:Fiducial_1mm_Mask2mm -> 0_RD_Fiducial:Fiducial_1mm_Mask2mm
- ID1: footprint RD-Symbols-Silkscreen:STACKUP_ID_2L -> 0_RD_Identification:STACKUP_ID_2L
- ID2: footprint RD-Symbols-Silkscreen:BOARD_IDENTIFICATION -> 0_RD_Identification:BOARD_IDENTIFICATION
- J1: footprint Connector_Molex_Addendum:Molex_Micro-Fit_3.0_43650-0215_1x02_P3.00mm_Vertical -> 0_Connector:Molex_KK-396_5273-02A_1x02_P3.96mm_Vertical
- J4: footprint Connector:Tag-Connect_TC2030-IDC-NL_2x03_P1.27mm_Vertical -> 0_RD_Testpoint:Tag-Connect_TC2030-IDC-NL_2x03_P1.27mm_Vertical
- J9: footprint Connector_Molex_Addendum:Molex_Micro-Fit_3.0_43650-0415_1x04_P3.00mm_Vertical -> 0_Connector:Molex_Micro-Fit_3.0_43650-0415_1x04_P3.00mm_Vertical
- JP3: footprint Jumpers:PinHeader_1x04_P2.54mm_Vertical -> 0_Jumper:PinHeader_1x04_P2.54mm_Vertical
- JP4: footprint Jumpers:PinHeader_2x04_P2.54mm_Vertical -> 0_Jumper:PinHeader_2x04_P2.54mm_Vertical
- R1, R10, R11, R13, R16, R17, R18, R19, R2, R20, R21, R22, R23, R24, R25, R26, R27, R28, R29, R3, R30, R31, R33, R34, R35, R36, R37, R39, R4, R40, R41, R42, R43, R44, R45, R46, R47, R48, R49, R5, R50, R51, R52, R53, R54, R55, R56, R6, R7, R8, R9: footprint Resistor_SMD:R_0603_1608Metric -> 0_RD_Resistor_SMD:R_0603_1608_DensityHigh
- R32: footprint Resistor_SMD:R_0603_1608Metric -> 0_RD_Resistor_SMD:R_0603_1608_DensityLow
- R38: footprint Resistor_SMD:R_0402_1005Metric -> 0_RD_Resistor_SMD:R_0402_1005_DensityHigh
- SW2, SW3: footprint PTS526SxxxSMTR2:SW_SPST_PTS526xxxSMTR -> 0_Switch_SMD:SW_SPST_PTS526xxxSMTR
- TP1: footprint RD-Testpoints:TestPoint_Pad_D1.0mm -> 0_RD_Testpoint:TestPoint_Pad_D1.0mm
- TP10: renamed from TP6; footprint RD-Testpoints:TestPoint_Pad_D0.4mm -> 0_RD_Testpoint:TestPoint_Pad_D0.4mm
- TP11: renamed from TP7; footprint RD-Testpoints:TestPoint_Pad_D0.4mm -> 0_RD_Testpoint:TestPoint_Pad_D0.4mm
- TP12: renamed from TP8; footprint RD-Testpoints:TestPoint_Pad_D0.4mm -> 0_RD_Testpoint:TestPoint_Pad_D0.4mm
- TP13: renamed from TP9; footprint RD-Testpoints:TestPoint_Pad_D0.4mm -> 0_RD_Testpoint:TestPoint_Pad_D0.4mm
- TP14: renamed from TP10; footprint RD-Testpoints:TestPoint_Pad_D1.0mm -> 0_RD_Testpoint:TestPoint_Pad_D1.0mm
- TP15: renamed from TP11; footprint RD-Testpoints:TestPoint_Pad_D1.0mm -> 0_RD_Testpoint:TestPoint_Pad_D1.0mm
- TP16: renamed from TP12; footprint RD-Testpoints:TestPoint_Pad_D0.4mm -> 0_RD_Testpoint:TestPoint_Pad_D0.4mm
- TP17: renamed from TP13; footprint RD-Testpoints:TestPoint_Pad_D0.4mm -> 0_RD_Testpoint:TestPoint_Pad_D0.4mm
- TP18: renamed from TP14; footprint RD-Testpoints:TestPoint_Pad_D1.0mm -> 0_RD_Testpoint:TestPoint_Pad_D1.0mm
- TP22: renamed from TP15; footprint RD-Testpoints:TestPoint_Pad_D0.4mm -> 0_RD_Testpoint:TestPoint_Pad_D0.4mm
- TP23: renamed from TP16; footprint RD-Testpoints:TestPoint_Pad_D0.4mm -> 0_RD_Testpoint:TestPoint_Pad_D0.4mm
- TP24: renamed from TP17; footprint RD-Testpoints:TestPoint_Pad_D0.4mm -> 0_RD_Testpoint:TestPoint_Pad_D0.4mm
- TP25: renamed from TP18; footprint RD-Testpoints:TestPoint_Pad_D0.4mm -> 0_RD_Testpoint:TestPoint_Pad_D0.4mm
- TP27: renamed from TP19; value GND -> G; footprint RD-Testpoints:TestPoint_Pad_1.0x1.0mm -> 0_RD_Testpoint:TestPoint_Pad_1.0x1.0mm
- TP28: renamed from TP20; value GND -> G; footprint RD-Testpoints:TestPoint_Pad_1.0x1.0mm -> 0_RD_Testpoint:TestPoint_Pad_1.0x1.0mm
- TP29: renamed from TP21; value GND -> G; footprint RD-Testpoints:TestPoint_Pad_1.0x1.0mm -> 0_RD_Testpoint:TestPoint_Pad_1.0x1.0mm
- TP3: renamed from TP2; footprint RD-Testpoints:TestPoint_Pad_D0.4mm -> 0_RD_Testpoint:TestPoint_Pad_D0.4mm
- TP30: renamed from TP22; value GND -> G; footprint RD-Testpoints:TestPoint_Pad_1.0x1.0mm -> 0_RD_Testpoint:TestPoint_Pad_1.0x1.0mm
- TP38: renamed from TP23; footprint RD-Testpoints:TestPoint_Pad_D0.4mm -> 0_RD_Testpoint:TestPoint_Pad_D0.4mm
- TP43: renamed from TP24; footprint RD-Testpoints:TestPoint_Pad_D0.4mm -> 0_RD_Testpoint:TestPoint_Pad_D0.4mm
- TP7: renamed from TP3; footprint RD-Testpoints:TestPoint_Pad_D1.0mm -> 0_RD_Testpoint:TestPoint_Pad_D1.0mm
- TP8: renamed from TP4; footprint RD-Testpoints:TestPoint_Pad_D1.0mm -> 0_RD_Testpoint:TestPoint_Pad_D1.0mm
- TP9: renamed from TP5; footprint RD-Testpoints:TestPoint_Pad_D0.4mm -> 0_RD_Testpoint:TestPoint_Pad_D0.4mm
- U5: footprint AP7362-33SP-13:SOIC-8-1EP_3.9x4.9mm_P1.27mm_EP2.6x3.5mm_ThermalVias -> 0_SOIC:SOIC-8-1EP_3.9x4.9mm_P1.27mm_EP2.6x3.5mm_ThermalVias
- moved TP28 29.2 mm to (195.5, 104.4)
- moved R22 14.7 mm to (232.1, 131.3)
- moved D3 14.7 mm to (231.6, 132.9)
- moved R23 11.9 mm to (223.1, 86.9), turned to 0 degrees
- moved TP24 11.3 mm to (229.0, 104.4)
- moved TP25 9.03 mm to (228.5, 105.7)
- moved TP15 7.93 mm to (215.3, 123.0)
- moved TP11 5.80 mm to (223.9, 178.6)
- moved R56 5.69 mm to (234.0, 91.0)
- moved C43 5.17 mm to (234.0, 103.7), turned to 0 degrees
- moved TP29 5.02 mm to (221.4, 151.2)
- moved TP23 4.55 mm to (200.6, 101.4)
- moved R55 4.52 mm to (234.0, 96.0)
- moved C23 4.30 mm to (198.5, 81.5), turned to 0 degrees
- moved C44 3.96 mm to (234.0, 98.6), turned to 0 degrees
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Connections:
- FB1 pad 2: +3V3 -> VDD
Routing:
- net +3V3: track 340.5 -> 104.8 mm, vias 9 -> 12
- net GND: track 78.8 -> 55.3 mm, vias 453 -> 362
- net /SYSTEM OVERVIEW/MICROCONTROLLER/CAN_H: track 13.0 -> 28.4 mm
- net /SYSTEM OVERVIEW/MICROCONTROLLER/CAN_120R_SW: track 11.6 -> 1.78 mm
- net +VM: track 30.4 -> 39.0 mm
- net /SYSTEM OVERVIEW/MICROCONTROLLER/BTN_N: track 22.1 -> 14.4 mm
- net VBUS: track 9.38 -> 3.40 mm
- net /SYSTEM OVERVIEW/MICROCONTROLLER/CAN_L: track 19.2 -> 25.0 mm
- net /SYSTEM OVERVIEW/MICROCONTROLLER/SW3_SIG: track 0.00 -> 5.64 mm
- net /SYSTEM OVERVIEW/MICROCONTROLLER/SW4_SIG: track 0.00 -> 5.64 mm
- net /SYSTEM OVERVIEW/MICROCONTROLLER/SW1_SIG: track 0.00 -> 5.64 mm
- net /SYSTEM OVERVIEW/MICROCONTROLLER/SW2_SIG: track 0.00 -> 5.64 mm
- net /SYSTEM OVERVIEW/POWER MANAGEMENT/BRAKE_SENSE: track 0.00 -> 5.06 mm
- net /SYSTEM OVERVIEW/MICROCONTROLLER/VM_ALERT_N: track 69.8 -> 73.8 mm
- net /SYSTEM OVERVIEW/MICROCONTROLLER/LED_YEL: track 7.78 -> 3.85 mm
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- added copper zone on B.Cu, net +3V3
- added copper zone on F.Cu, net /SYSTEM OVERVIEW/MICROCONTROLLER/BTN_N
- removed copper zone on F.Cu, net /SYSTEM OVERVIEW/MICROCONTROLLER/SW1_SIG
- removed copper zone on F.Cu, net /SYSTEM OVERVIEW/MICROCONTROLLER/SW2_SIG
- removed copper zone on F.Cu, net /SYSTEM OVERVIEW/MICROCONTROLLER/SW3_SIG
- removed copper zone on F.Cu, net /SYSTEM OVERVIEW/MICROCONTROLLER/SW4_SIG
- removed copper zone on F.Cu, net /SYSTEM OVERVIEW/POWER MANAGEMENT/BRAKE_SENSE
Other:
- board text added: "+VIN"
- board text added: "3V3"
- board text added: "CS"
- board text added: "ERROR"
- board text added: "G"
- board text added: "H"
- board text added: "HB"
- board text added: "IN"
- board text added: "L"
- board text added: "MISO"
- board text added: "MOSI"
- board text added: "RX"
- board text added: "SCK"
- board text added: "SCL"
- board text added: "SDA"
- board text added: "TX"
- board text removed: "ADC"
- board text removed: "CAN"
- board text removed: "ENCODER"
- board text removed: "I2C"
- board text removed: "LED1"
- board text removed: "LED2"
- board text removed: "MOTOR"
- board text removed: "UART"
- board text removed: "VIN"

Commit message: chore(pcb): update project files
Routing:
- net /SYSTEM OVERVIEW/MOTOR CONTROL AND IO/DRV_CS: track 26.3 -> 25.8 mm
Other:
- board text removed: "MOTOR DRIVER"
- board text removed: "SWITCHES"
