File: project.kicad_sch (KiCad schematic)
At the start: 168 parts, among them J1 VIN_CONN, J10 SW2_CONN, J11 CAN_CONN, J12 I2C_CONN, J13 SW3_CONN, J14 ST-LINK_CONN, J15 TEMP_CONN, J16 AUX_ADC_CONN, J17 TAG_CONN, J18 SW4_CONN, J2 MOT_CONN, J3 DRV_DIAG, J4 DRV_SKT_LEFT, J5 DRV_SKT_RIGHT, J6 USB_CONN, J7 ENC_CONN, J8 SW1_CONN, J9 UART_CONN, Q1 UTT18P10L-TN3-R, Q2 NCE0106R, SW1 SW_RESET, SW2 SW_CAN_TERM, SW3 SW_USER, U1 LMR36510ADDAR, U2 TMC5160T Pro, U3 AP7362-33SP-13, U4 TLV6700QDDCRQ1, U5 INA238AIDGSR, U6 STM32L476RGT6, U7 TLV4041R5DBVR, U8 TJA1051T-3-1J-TD, U9 USBLC6-2SC6, Y1 ECS-80-8-30-JGN-TR, Y2 ECS-.327-6-34R-TR

Commit message: chore(template): update project files
Parts:
- added ID2: BOARD_IDENTIFICATION_MARKER, RD-Symbols-Silkscreen:BOARD_IDENTIFICATION, symbol Ryan-Dynamics:BOARD_IDENTIFICATION_MARKER
- J16: value AUX_ADC_CONN -> ADC_CONN
Other:
- moved on the sheet: ID1

Commit message: chore(pcb): update project files
Parts:
- J1: footprint Connector_Molex:Molex_Micro-Fit_3.0_43650-0215_1x02_P3.00mm_Vertical -> Connector_Molex_Addendum:Molex_Micro-Fit_3.0_43650-0215_1x02_P3.00mm_Vertical
- J2: footprint Connector_Molex:Molex_Micro-Fit_3.0_43650-0415_1x04_P3.00mm_Vertical -> Connector_Molex_Addendum:Molex_Micro-Fit_3.0_43650-0415_1x04_P3.00mm_Vertical
- Q1: value UTT18P10L-TN3-R -> CRTD700P10L; LCSC_PN C84900 -> C841381; MPN UTT18P10L-TN3-R -> CRTD700P10L; Manufacturer UTC -> CRMICRO; SPN C84900 -> C841381
Changed lines of the file:
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@@
 			)
 		)
-		(property "Footprint" "Connector_Molex:Molex_Micro-Fit_3.0_43650-0415_1x04_P3.00mm_Vertical"
+		(property "Footprint" "Connector_Molex_Addendum:Molex_Micro-Fit_3.0_43650-0415_1x04_P3.00mm_Vertical"
 			(at 745.49 99.06 0)
 			(effects
@@
 			)
 		)
+		(property "V_max" ""
+			(at 745.49 99.06 0)
+			(effects
+				(font
+					(size 1.27 1.27)
+				)
+				(hide yes)
+			)
+		)
+		(property "Tolerance" ""
+			(at 745.49 99.06 0)
+			(effects
+				(font
+					(size 1.27 1.27)
+				)
+				(hide yes)
+			)
+		)
+		(property "P_max" ""
+			(at 745.49 99.06 0)
+			(effects
+				(font
+					(size 1.27 1.27)
+				)
+				(hide yes)
+			)
+		)
+		(property "I_peak" ""
+			(at 745.49 99.06 0)
+			(effects
+				(font
+					(size 1.27 1.27)
+				)
+				(hide yes)
+			)
+		)
+		(property "Lifetime" ""
+			(at 745.49 99.06 0)
+			(effects
+				(font
+					(size 1.27 1.27)
+				)
+				(hide yes)
+			)
+		)
+		(property "Dielectric" ""
+			(at 745.49 99.06 0)
+			(effects
+				(font
+					(size 1.27 1.27)
+				)
+				(hide yes)
+			)
+		)
 		(pin "1"
 		)
@@
 			)
 		)
-		(property "Footprint" "Connector_Molex:Molex_Micro-Fit_3.0_43650-0215_1x02_P3.00mm_Vertical"
+		(property "Footprint" "Connector_Molex_Addendum:Molex_Micro-Fit_3.0_43650-0215_1x02_P3.00mm_Vertical"
 			(at 73.66 68.58 0)
 			(effects
@@
 			)
 		)
+		(property "V_max" ""
+			(at 73.66 68.58 0)
+			(effects
+				(font
+					(size 1.27 1.27)
+				)
+				(hide yes)
+			)
+		)
+		(property "Tolerance" ""
+			(at 73.66 68.58 0)
+			(effects
+				(font
+					(size 1.27 1.27)
+				)
+				(hide yes)
+			)
+		)
+		(property "P_max" ""
+			(at 73.66 68.58 0)
+			(effects
+				(font
+					(size 1.27 1.27)
+				)
+				(hide yes)
+			)
+		)
+		(property "I_peak" ""
+			(at 73.66 68.58 0)
+			(effects
+				(font
+					(size 1.27 1.27)
+				)
+				(hide yes)
+			)
+		)
+		(property "Lifetime" ""
+			(at 73.66 68.58 0)
+			(effects
+				(font
+					(size 1.27 1.27)
+				)
+				(hide yes)
+			)
+		)
+		(property "Dielectric" ""
+			(at 73.66 68.58 0)
+			(effects
+				(font
+					(size 1.27 1.27)
+				)
+				(hide yes)
+			)
+		)
 		(pin "2"
 		)
@@
 			)
 		)
-		(property "Value" "UTT18P10L-TN3-R"
+		(property "Value" "CRTD700P10L"
 			(at 130.81 64.77 90)
 			(effects
@@
 			)
 		)
-		(property "Datasheet" "https://www.lcsc.com/datasheet/C84900.pdf"
+		(property "Datasheet" "https://www.lcsc.com/datasheet/C841381.pdf"
 			(at 130.81 71.12 0)
 			(effects
@@
 			)
 		)
-		(property "Description" "MOSFET P-CH 100V 18A TO-252"
+		(property "Description" "MOSFET P-CH 100V-26A TO-252"
 			(at 130.81 71.12 0)
 			(effects
@@
 			)
 		)
-		(property "Manufacturer" "UTC"
+		(property "Manufacturer" "CRMICRO"
 			(at 130.81 71.12 90)
 			(effects
@@
 			)
 		)
-		(property "MPN" "UTT18P10L-TN3-R"
+		(property "MPN" "CRTD700P10L"
 			(at 130.81 71.12 90)
 			(effects
@@
 			)
 		)
-		(property "LCSC_PN" "C84900"
+		(property "LCSC_PN" "C841381"
 			(at 130.81 71.12 90)
 			(effects
@@
 			)
 		)
-		(property "SPN" "C84900"
+		(property "SPN" "C841381"
 			(at 130.81 71.12 90)
 			(effects
@@
 			(effects
 				(font
+					(size 1.27 1.27)
+				)
+				(hide yes)
+			)
+		)
+		(property "V_max" ""
+			(at 130.81 71.12 0)
+			(effects
+				(font
+					(size 1.27 1.27)
+				)
+				(hide yes)
+			)
+		)
+		(property "Tolerance" ""
+			(at 130.81 71.12 0)
+			(effects
+				(font
+					(size 1.27 1.27)
+				)
+				(hide yes)
+			)
+		)
+		(property "P_max" ""
+			(at 130.81 71.12 0)
+			(effects
+				(font
+					(size 1.27 1.27)
+				)
+				(hide yes)
+			)
+		)
+		(property "I_peak" ""
+			(at 130.81 71.12 0)
+			(effects
+				(font
+					(size 1.27 1.27)
+				)
+				(hide yes)
+			)
+		)
+		(property "Lifetime" ""
+			(at 130.81 71.12 0)
+			(effects
+				(font
+					(size 1.27 1.27)
+				)
+				(hide yes)
+			)
+		)
+		(property "Dielectric" ""
+			(at 130.81 71.12 0)
+			(effects
+				(font

Commit message: chore(pcb): update project files
Parts:
- C1, C10, C11, C12, C16, C17, C18, C19, C25, C26, C35, C37, C38, C39, C40, C41, C42, C43, C44, C45, C46, C8: LCSC_PN C14663 -> (none); SPN2 (none) -> C14663; Supplier2 (none) -> LCSC
- C13, C31, C32: LCSC_PN C57112 -> (none); MPN 0603B103K500NT -> CC0603KRX7R9BB103; MPN2 (none) -> 0603B103K500NT; Manufacturer FH (Guangdong Fenghua Advanced Tech) -> YAGEO; Manufacturer2 (none) -> FH (Guangdong Fenghua Advanced Tech); SPN C57112 -> 311-1085-1-ND; SPN2 (none) -> C57112; Supplier LCSC -> DigiKey; Supplier2 (none) -> LCSC
- C14, C15, C20: LCSC_PN C28323 -> (none); MPN CL21B105KBFNNNE -> CC0805MKX7R6BB105; MPN2 (none) -> CL21B105KBFNNNE; Manufacturer Samsung Electro-Mechanics -> YAGEO; Manufacturer2 (none) -> Samsung Electro-Mechanics; SPN 1276-1029-1-ND -> 311-3431-1-ND; SPN2 (none) -> C28323; Supplier2 (none) -> LCSC; Voltage_Rating 50V -> 10V
- C2: LCSC_PN C2839509 -> (none); SPN2 (none) -> C2839509; Supplier2 (none) -> LCSC
- C21: LCSC_PN C113803 -> (none); SPN2 (none) -> C113803; Supplier2 (none) -> LCSC
- C22: LCSC_PN C70463 -> (none); SPN2 (none) -> C70463; Supplier2 (none) -> LCSC
- C23: LCSC_PN C88774 -> (none); SPN2 (none) -> C88774; Supplier Digikey -> DigiKey; Supplier2 (none) -> LCSC
- C24, C27: value 10p -> 30p; LCSC_PN C1634 -> (none); MPN CL10C100JB8NNNC -> CC0603JRNPO9BN300; MPN2 (none) -> 0603CG300J500NT; Manufacturer Samsung Electro-Mechanics -> YAGEO; Manufacturer2 (none) -> FH (Guangdong Fenghua Advanced Tech); SPN 1276-1027-1-ND -> 311-3357-1-ND; SPN2 (none) -> C1658; Supplier Digikey -> DigiKey; Supplier2 (none) -> LCSC
- C28, C29, C30, C36: footprint Capacitor_SMD:C_0603_1608Metric -> Capacitor_SMD:C_0805_2012Metric; Dielectric X5R -> X7R; LCSC_PN C19702 -> (none); MPN CL10A106KP8NNNC -> CC0805KFX7R6BB106; MPN2 (none) -> CL10A106KP8NNNC; Manufacturer Samsung Electro-Mechanics -> YAGEO; Manufacturer2 (none) -> Samsung Electro-Mechanics; SPN 1276-1192-1-ND -> 13-CC0805KFX7R6BB106CT-ND; SPN2 (none) -> C19702; Supplier Digikey -> DigiKey; Supplier2 (none) -> LCSC
- C3, C4: LCSC_PN C577211 -> (none); SPN2 (none) -> C577211; Supplier2 (none) -> LCSC
- C33, C34: value 10p -> 15p; LCSC_PN C32949 -> (none); MPN CL05C100JB5NNNC -> CC0402JRNPO9BN150; MPN2 (none) -> 0402CG150J500NT; Manufacturer Samsung Electro-Mechanics -> YAGEO; Manufacturer2 (none) -> FH (Guangdong Fenghua Advanced Tech); SPN 1276-1139-1-ND -> 311-1017-1-ND; SPN2 (none) -> C1548; Supplier Digikey -> DigiKey; Supplier2 (none) -> LCSC
- C5: LCSC_PN C113892 -> (none); SPN2 (none) -> C113892; Supplier2 (none) -> LCSC
- C6, C7: LCSC_PN C110045 -> (none); SPN2 (none) -> C110045; Supplier2 (none) -> LCSC
- C9: LCSC_PN C29823 -> (none); MPN 1206B475K500NT -> CC1206KFX7R9BB475; MPN2 (none) -> 1206B475K500NT; Manufacturer FH (Guangdong Fenghua Advanced Tech) -> YAGEO; Manufacturer2 (none) -> FH (Guangdong Fenghua Advanced Tech); SPN C29823 -> 13-CC1206KFX7R9BB475CT-ND; SPN2 (none) -> C29823; Supplier LCSC -> DigiKey; Supplier2 (none) -> LCSC
- D1: LCSC_PN C85383 -> (none); SPN2 (none) -> C85383; Supplier2 (none) -> LCSC
- D2, D3: LCSC_PN C2297 -> (none); MPN KT-0805G -> LTST-C171KGKT; MPN2 (none) -> KT-0805G; Manufacturer Hubei KENTO Elec -> Lite-On Inc.; Manufacturer2 (none) -> Hubei KENTO Elec; SPN C2297 -> 160-1426-1-ND; SPN2 (none) -> C2297; Supplier LCSC -> DigiKey; Supplier2 (none) -> LCSC
- D5: LCSC_PN C75176 -> (none); SPN2 (none) -> C75176; Supplier2 (none) -> LCSC
- D6: LCSC_PN C2296 -> (none); MPN KT-0805Y -> LTST-C171YKT; MPN2 (none) -> KT-0805Y; Manufacturer Hubei KENTO Elec -> Lite-On Inc.; Manufacturer2 (none) -> Hubei KENTO Elec; SPN C2296 -> 160-1431-1-ND; SPN2 (none) -> C2296; Supplier LCSC -> DigiKey; Supplier2 (none) -> LCSC
- D7: LCSC_PN C84256 -> (none); MPN NCD0805R1 -> LTST-C171KRKT; MPN2 (none) -> NCD0805R1; Manufacturer NATIONSTAR -> Lite-On Inc.; Manufacturer2 (none) -> NATIONSTAR; SPN C84256 -> 160-1427-1-ND; SPN2 (none) -> C84256; Supplier LCSC -> DigiKey; Supplier2 (none) -> LCSC
- F1: LCSC_PN C12604 -> (none); SPN2 (none) -> C12604; Supplier2 (none) -> LCSC
- FB1: LCSC_PN C14709 -> (none); SPN2 (none) -> C14709; Supplier2 (none) -> LCSC
- FH1: value XF-508P-B-B -> VIN_FH; LCSC_PN C19727305 -> (none); MPN XF-508P-B-B -> 3568; MPN2 (none) -> XF-508P-B-B; Manufacturer XFCN -> Keystone Electronics; Manufacturer2 (none) -> XFCN; SPN C19727305 -> 36-3568-ND; SPN2 (none) -> C19727305; Supplier LCSC -> DigiKey; Supplier2 (none) -> LCSC
- J1: LCSC_PN C239439 -> (none); MPN C3030WV-2P -> 0436500215; MPN2 (none) -> C3030WV-2P; Manufacturer CJT(Changjiang Connectors) -> Molex; Manufacturer2 (none) -> CJT(Changjiang Connectors); SPN C239439 -> WM1917-ND; SPN2 (none) -> C239439; Supplier LCSC -> DigiKey; Supplier2 (none) -> LCSC
- J10, J13, J18, J8, JP4: LCSC_PN C32713269 -> (none); MPN HX PZ2.54-1x3P ZZ -> HM3212; MPN2 (none) -> HX PZ2.54-1x3P ZZ; Manufacturer hanxia -> Jaycar Electronics; Manufacturer2 (none) -> hanxia; SPN C32713269 -> HM3212; SPN2 (none) -> C32713269; Supplier LCSC -> Jaycar Electronics; Supplier2 (none) -> LCSC
- J11, J16: LCSC_PN C239363 -> (none); MPN A2543WV-3P -> HM3413; MPN2 (none) -> A2543WV-3P; Manufacturer CJT(Changjiang Connectors) -> Jaycar Electronics; Manufacturer2 (none) -> CJT(Changjiang Connectors); SPN C239363 -> HM3413; SPN2 (none) -> C239363; Supplier LCSC -> Jaycar Electronics; Supplier2 (none) -> LCSC
- J12, J9: LCSC_PN C239364 -> (none); MPN A2543WV-4P -> HM3414; MPN2 (none) -> A2543WV-4P; Manufacturer CJT(Changjiang Connectors) -> Jaycar Electronics; Manufacturer2 (none) -> CJT(Changjiang Connectors); SPN C239364 -> HM3414; SPN2 (none) -> C239364; Supplier LCSC -> Jaycar Electronics; Supplier2 (none) -> LCSC
- J14: LCSC_PN C27985148 -> (none); MPN HC-PZ127-7.2L-2x7PS -> 20021121-00014T1LF; MPN2 (none) -> HC-PZ127-7.2L-2x7PS; Manufacturer Hong Cheng -> Amphenol ICC (FCI); Manufacturer2 (none) -> Hong Cheng; SPN C27985148 -> 20021121-00014T1LF-ND; SPN2 (none) -> C27985148; Supplier LCSC -> DigiKey; Supplier2 (none) -> LCSC
- J15: LCSC_PN C239362 -> (none); MPN A2543WV-2P -> HM3412; MPN2 (none) -> A2543WV-2P; Manufacturer CJT(Changjiang Connectors) -> Jaycar Electronics; Manufacturer2 (none) -> CJT(Changjiang Connectors); SPN C239362 -> HM3412; SPN2 (none) -> C239362; Supplier LCSC -> Jaycar Electronics; Supplier2 (none) -> LCSC
- J2: LCSC_PN C239441 -> (none); MPN C3030WV-4P -> 0436500415; MPN2 (none) -> C3030WV-4P; Manufacturer CJT(Changjiang Connectors) -> Molex; Manufacturer2 (none) -> CJT(Changjiang Connectors); SPN C239441 -> WM1919-ND; SPN2 (none) -> C239441; Supplier LCSC -> DigiKey; Supplier2 (none) -> LCSC
- J3: LCSC_PN C41427517 -> (none)
- J4, J5: LCSC_PN C41427523 -> (none)
- J6: LCSC_PN C2894897 -> (none); MPN HC-TYPE-C-16P-01A -> USB4105-GF-A; MPN2 (none) -> HC-TYPE-C-16P-01A; Manufacturer HCTL -> GCT; Manufacturer2 (none) -> HCTL; SPN C2894897 -> 2073-USB4105-GF-ACT-ND; SPN2 (none) -> C2894897; Supplier LCSC -> DigiKey; Supplier2 (none) -> LCSC
- J7: LCSC_PN C239366 -> (none); MPN A2543WV-6P -> HM3416; MPN2 (none) -> A2543WV-6P; Manufacturer CJT(Changjiang Connectors) -> Jaycar Electronics; Manufacturer2 (none) -> CJT(Changjiang Connectors); SPN C239366 -> HM3416; SPN2 (none) -> C239366; Supplier LCSC -> Jaycar Electronics; Supplier2 (none) -> LCSC
- JP1: LCSC_PN C32713277 -> (none); MPN HX PZ2.54-2x4P ZZ -> HM3250; MPN2 (none) -> HX PZ2.54-2x4P ZZ; Manufacturer hanxia -> Jaycar Electronics; Manufacturer2 (none) -> hanxia; SPN C32713277 -> HM3250; SPN2 (none) -> C32713277; Supplier LCSC -> Jaycar Electronics; Supplier2 (none) -> LCSC
- JP2: LCSC_PN C32713270 -> (none); MPN HX PZ2.54-1x4P ZZ -> HM3212; MPN2 (none) -> HX PZ2.54-1x4P ZZ; Manufacturer hanxia -> Jaycar Electronics; Manufacturer2 (none) -> hanxia; SPN C32713270 -> HM3212; SPN2 (none) -> C32713270; Supplier LCSC -> Jaycar Electronics; Supplier2 (none) -> LCSC
- L1: LCSC_PN C54620267 -> (none); MPN APV ANR8040T270M -> ASPI-8040S-270M-T; MPN2 (none) -> ANR8040T270M; Manufacturer APV -> Abracon LLC; Manufacturer2 (none) -> APV; SPN C54620267 -> ASPI-8040S-270M-TCT-ND; SPN2 (none) -> C54620267; Supplier LCSC -> DigiKey; Supplier2 (none) -> LCSC
- Q1: LCSC_PN C841381 -> (none); MPN CRTD700P10L -> MCU055P10-TP; MPN2 (none) -> CRTD700P10L; Manufacturer CRMICRO -> MCC (Micro Commercial Components); Manufacturer2 (none) -> CRMICRO; SPN C841381 -> 353-MCU055P10-TPCT-ND; SPN2 (none) -> C841381; Supplier LCSC -> DigiKey; Supplier2 (none) -> LCSC
- Q2: LCSC_PN C189607 -> (none); MPN NCE0106R -> SL10N10A; MPN2 (none) -> NCE0106R; Manufacturer NCE -> Shenzhen Slkormicro Semicon Co., Ltd.; Manufacturer2 (none) -> NCE; SPN C189607 -> 5399-SL10N10ACT-ND; SPN2 (none) -> C189607; Supplier LCSC -> DigiKey; Supplier2 (none) -> LCSC
- R1: LCSC_PN C1711510 -> (none); SPN C1711510 -> 541-WSL10202L000FEACT-ND; SPN2 (none) -> C1711510; Supplier LCSC -> DigiKey; Supplier2 (none) -> LCSC
- R10, R39, R40, R9: LCSC_PN C22859 -> (none); MPN 0603WAF100JT5E -> RT0603FRE1310RL; MPN2 (none) -> 0603WAF100JT5E; Manufacturer UNI-ROYAL -> YAGEO; Manufacturer2 (none) -> UNI-ROYAL; SPN C22859 -> 13-RT0603FRE1310RLCT-ND; SPN2 (none) -> C22859; Supplier LCSC -> DigiKey; Supplier2 (none) -> LCSC
- R11, R13, R14, R19, R35, R41, R42, R44, R5, R54, R55: LCSC_PN C25804 -> (none); MPN 0603WAF1002T5E -> RT0603FRE1010KL; MPN2 (none) -> 0603WAF1002T5E; Manufacturer UNI-ROYAL -> YAGEO; Manufacturer2 (none) -> UNI-ROYAL; SPN C25804 -> 13-RT0603FRE1010KLCT-ND; SPN2 (none) -> C25804; Supplier LCSC -> DigiKey; Supplier2 (none) -> LCSC
- R12, R27: LCSC_PN C2989464 -> (none); MPN TC0325B1004T5F -> RT0603BRD071ML; MPN2 (none) -> TC0325B1004T5F; Manufacturer UNI-ROYAL -> YAGEO; Manufacturer2 (none) -> UNI-ROYAL; SPN C2989464 -> YAG4498CT-ND; SPN2 (none) -> C2989464; Supplier LCSC -> DigiKey; Supplier2 (none) -> LCSC; Voltage_Rating (none) -> 75V
- R15: LCSC_PN C21189 -> (none); MPN 0603WAF0000T5E -> RC0402JR-070RP; MPN2 (none) -> 0402WGF0000TCE; Manufacturer UNI-ROYAL -> YAGEO; Manufacturer2 (none) -> UNI-ROYAL; Power_Rating 1/10W -> 1/16W; SPN C21189 -> YAG1279CT-ND; SPN2 (none) -> C17168; Supplier LCSC -> DigiKey; Supplier2 (none) -> LCSC
- R16, R17, R21, R22, R23, R24, R4, R45, R52, R53: LCSC_PN C21190 -> (none); MPN 0603WAF1001T5E -> RT0603FRE071KL; MPN2 (none) -> 0603WAF1001T5E; Manufacturer UNI-ROYAL -> YAGEO; Manufacturer2 (none) -> UNI-ROYAL; SPN C21190 -> YAG2323CT-ND; SPN2 (none) -> C21190; Supplier LCSC -> DigiKey; Supplier2 (none) -> LCSC
- R18: LCSC_PN C2989227 -> (none); MPN TC0350B4301T5F -> RT0603BRD074K32L; MPN2 (none) -> TC0350B4301T5F; Manufacturer UNI-ROYAL -> YAGEO; Manufacturer2 (none) -> UNI-ROYAL; SPN C2989227 -> YAG4567CT-ND; SPN2 (none) -> C2989227; Supplier LCSC -> DigiKey; Supplier2 (none) -> LCSC; Voltage_Rating (none) -> 75V
- R2, R30, R6, R8: LCSC_PN C25803 -> (none); MPN 0603WAF1003T5E -> RT0603FRE07100KL; MPN2 (none) -> 0603WAF1003T5E; Manufacturer UNI-ROYAL -> YAGEO; Manufacturer2 (none) -> UNI-ROYAL; SPN C25803 -> YAG2319CT-ND; SPN2 (none) -> C25803; Supplier LCSC -> DigiKey; Supplier2 (none) -> LCSC
- R20: LCSC_PN C517416 -> (none); MPN TC0325B9101T5H -> RT0603BRD079K1L; Manufacturer UNI-ROYAL -> YAGEO; Power_Rating 167mW -> 1/10W; SPN C517416 -> YAG1756CT-ND; SPN2 (none) -> C861612; Supplier LCSC -> DigiKey; Supplier2 (none) -> LCSC
- R25, R26: LCSC_PN C2992638 -> (none); MPN CUH2512J150RE04Z -> RPCQ2512JT150R; MPN2 (none) -> CUH2512J150RE04Z; Manufacturer EVER OHMS -> Stackpole Electronics Inc; Manufacturer2 (none) -> EVER OHMS; Notes (none) -> Pulse rating required.; Power_Rating 3W -> 4W; SPN C2992638 -> 738-RPCQ2512JT150RCT-ND; SPN2 (none) -> C2992638; Supplier LCSC -> DigiKey; Supplier2 (none) -> LCSC
- R28: LCSC_PN C22775 -> (none); MPN 0603WAF1000T5E -> RT0603FRE07100RL; MPN2 (none) -> 0603WAF1000T5E; Manufacturer UNI-ROYAL -> YAGEO; Manufacturer2 (none) -> UNI-ROYAL; SPN C22775 -> YAG2320CT-ND; SPN2 (none) -> C22775; Supplier LCSC -> DigiKey; Supplier2 (none) -> LCSC
- R29: LCSC_PN C2988916 -> (none); MPN TC0325B1102T5F -> RT0603BRD0711KL; MPN2 (none) -> TC0325B1102T5F; Manufacturer UNI-ROYAL -> YAGEO; Manufacturer2 (none) -> UNI-ROYAL; SPN C2988916 -> YAG1511CT-ND; SPN2 (none) -> C2988916; Supplier LCSC -> DigiKey; Supplier2 (none) -> LCSC
- R3: LCSC_PN C13167 -> (none); MPN 0603WAF2701T5E -> RT0603FRE072K7L; MPN2 (none) -> 0603WAF2701T5E; Manufacturer UNI-ROYAL -> YAGEO; Manufacturer2 (none) -> UNI-ROYAL; SPN C13167 -> YAG5955CT-ND; SPN2 (none) -> C13167; Supplier LCSC -> DigiKey; Supplier2 (none) -> LCSC
- R31, R32, R33, R34: LCSC_PN C23162 -> (none); MPN 0603WAF4701T5E -> RT0603FRE074K7L; MPN2 (none) -> 0603WAF4701T5E; Manufacturer UNI-ROYAL -> YAGEO; Manufacturer2 (none) -> UNI-ROYAL; SPN C23162 -> YAG1238CT-ND; SPN2 (none) -> C23162; Supplier LCSC -> DigiKey; Supplier2 (none) -> LCSC
- R36: LCSC_PN C22787 -> (none); MPN 0603WAF1200T5E -> RT0603FRE07120RL; MPN2 (none) -> 0603WAF1200T5E; Manufacturer UNI-ROYAL -> YAGEO; Manufacturer2 (none) -> UNI-ROYAL; SPN C22787 -> 13-RT0603FRE07120RLCT-ND; SPN2 (none) -> C22787; Supplier LCSC -> DigiKey; Supplier2 (none) -> LCSC
- R37, R38: LCSC_PN C23186 -> (none); MPN 0603WAF5101T5E -> RT0603FRD075K1L; MPN2 (none) -> 0603WAF5101T5E; Manufacturer UNI-ROYAL -> YAGEO; Manufacturer2 (none) -> UNI-ROYAL; SPN C23186 -> 13-RT0603FRD075K1LCT-ND; SPN2 (none) -> C23186; Supplier LCSC -> DigiKey; Supplier2 (none) -> LCSC
- R43, R46, R47, R48, R50, R51: LCSC_PN C23345 -> (none); MPN 0603WAF220JT5E -> RT0603FRE0722RL; MPN2 (none) -> 0603WAF220JT5E; Manufacturer UNI-ROYAL -> YAGEO; Manufacturer2 (none) -> UNI-ROYAL; SPN C23345 -> YAG5950CT-ND; SPN2 (none) -> C23345; Supplier LCSC -> DigiKey; Supplier2 (none) -> LCSC
- R49: LCSC_PN C25819 -> (none); MPN 0603WAF4702T5E -> RT0603FRE0747KL; MPN2 (none) -> 0603WAF4702T5E; Manufacturer UNI-ROYAL -> YAGEO; Manufacturer2 (none) -> UNI-ROYAL; SPN C25819 -> YAG3355CT-ND; SPN2 (none) -> C25819; Supplier LCSC -> DigiKey; Supplier2 (none) -> LCSC
- R7: LCSC_PN C25962 -> (none); MPN 0603WAF2492T5E -> RT0603FRE0724K9L; MPN2 (none) -> 0603WAF2492T5E; Manufacturer UNI-ROYAL -> YAGEO; Manufacturer2 (none) -> UNI-ROYAL; SPN C25962 -> YAG5951CT-ND; SPN2 (none) -> C25962; Supplier LCSC -> DigiKey; Supplier2 (none) -> LCSC
- SW1, SW3: LCSC_PN C2689521 -> (none); SPN2 (none) -> C2689521; Supplier2 (none) -> LCSC
- SW2: LCSC_PN C5299502 -> (none); MPN SMQS-01R-TP -> DS01-254-L-01BE; MPN2 (none) -> SMQS-01R-TP; Manufacturer SM Switch -> Same Sky (Formerly CUI Devices); Manufacturer2 (none) -> SM Switch; SPN C5299502 -> DS01-254-L-01BE; SPN2 (none) -> C5299502; Supplier LCSC -> DigiKey; Supplier2 (none) -> LCSC
- U1: LCSC_PN C1858393 -> (none); SPN2 (none) -> C1858393; Supplier2 (none) -> LCSC
- U2: SPN TMC5160T Pro -> 1050000063; Supplier BIGTREETECH -> DREMC
- U3: LCSC_PN C780775 -> (none); SPN2 (none) -> C780775; Supplier2 (none) -> LCSC
- U4: LCSC_PN C2870089 -> (none); SPN2 (none) -> C2870089; Supplier2 (none) -> LCSC
- U5: LCSC_PN C2868250 -> (none); SPN2 (none) -> C2868250; Supplier2 (none) -> LCSC
- U6: LCSC_PN C74797 -> (none); SPN2 (none) -> C74797; Supplier2 (none) -> LCSC
- U7: LCSC_PN C2873273 -> (none); SPN2 (none) -> C2873273; Supplier2 (none) -> LCSC
- U8: value TJA1051T-3-1J-TD -> TJA1051T/3; LCSC_PN C51954344 -> (none); MPN TJA1051T-3-1J-TD -> TJA1051T/3,118; MPN2 (none) -> TJA1051T-3-1J-TD; Manufacturer TDSEMIC -> NXP USA Inc.; Manufacturer2 (none) -> TDSEMIC; SPN C51954344 -> 568-8684-1-ND; SPN2 (none) -> C51954344; Supplier LCSC -> DigiKey; Supplier2 (none) -> LCSC
- U9: LCSC_PN C2687116 -> (none); MPN2 (none) -> USBLC6-2SC6; Manufacturer UMW -> STMicroelectronics; Manufacturer2 (none) -> UMW; SPN C2687116 -> 497-5235-1-ND; SPN2 (none) -> C2687116; Supplier LCSC -> DigiKey; Supplier2 (none) -> LCSC
- Y1: value ECS-80-8-30-JGN-TR -> X50328MSB2GI; C_L 8pF -> 20pF; MPN ECS-80-8-30-JGN-TR -> ECS-80-18-30-JGN-TR; MPN2 (none) -> X50328MSB2GI; Manufacturer2 (none) -> YXC Crystal Oscillators; SPN 50-ECS-80-8-30-JGN-TRCT-ND -> XC2103CT-ND; SPN2 (none) -> C115962; Supplier2 (none) -> LCSC
- Y2: value ECS-.327-6-34R-TR -> Q13FC13500004; C_L 6pF -> 12.5pF; MPN ECS-.327-6-34R-TR -> ECS-.327-12.5-34B-TR; MPN2 (none) -> Q13FC13500004; Manufacturer2 (none) -> EPSON; SPN 50-ECS-.327-6-34R-TRCT-ND -> 50-ECS-.327-12.5-34B-TRCT-ND; SPN2 (none) -> C32346; Supplier2 (none) -> LCSC
Connections:
- net GND: now also C27.1, C34.1; no longer C27.2, C34.2
- net OSC32_OUT: now also C34.2; no longer C34.1
- net XTAL: now also C27.2; no longer C27.1

Commit message: chore(pcb): update project files
Parts:
- added C47: 10n, Capacitor_SMD:C_0603_1608Metric, symbol Device:C
- added R55: 1k, Resistor_SMD:R_0603_1608Metric, symbol Device:R
- added TP10: TEMP_ADC, RD-Testpoints:TestPoint_Pad_D0.4mm, symbol Connector:TestPoint
- added TP13: AUX_ADC, RD-Testpoints:TestPoint_Pad_D0.4mm, symbol Connector:TestPoint
- added TP6: ~{VM_UV}, RD-Testpoints:TestPoint_Pad_D0.4mm, symbol Connector:TestPoint
- added TP7: ~{VM_OV}, RD-Testpoints:TestPoint_Pad_D0.4mm, symbol Connector:TestPoint
- added TP8: ~{VM_ALERT}, RD-Testpoints:TestPoint_Pad_D0.4mm, symbol Connector:TestPoint
- renumbered R55 to R56, TP7 to TP11, TP8 to TP12, TP6 to TP9
Connections:
- net AUX_ADC: now also C47.2, R55.2, TP13.1; no longer J16.3 (Pin_3)
- net GND: now also C47.1
- net TEMP_ADC: now also TP10.1
- net ~{VM_ALERT}: now also TP8.1
- net ~{VM_OV}: now also TP7.1
- net ~{VM_UV}: now also TP6.1
- new net AUX_ADC_CONN: J16.3 (Pin_3), R55.1

Commit message: chore(pcb): update project files
Parts:
- added TP13: GND, RD-Testpoints:TestPoint_Pad_1.0x1.0mm, symbol Connector:TestPoint
- renumbered TP13 to TP14
Connections:
- net GND: now also TP13.1
Changed lines of the file:
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@@
 	)
 	(junction
+		(at 226.06 416.56)
+		(diameter 0)
+		(color 0 0 0 0)
+	)
+	(junction
 		(at 255.27 416.56)
 		(diameter 0)
@@
 	(wire
 		(pts
-			(xy 223.52 416.56) (xy 229.87 416.56)
+			(xy 223.52 416.56) (xy 226.06 416.56)
 		)
 		(stroke
@@
 	(wire
 		(pts
+			(xy 226.06 416.56) (xy 229.87 416.56)
+		)
+		(stroke
+			(width 0)
+			(type default)
+		)
+	)
+	(wire
+		(pts
 			(xy 506.73 73.66) (xy 506.73 76.2)
 		)
@@
 	(wire
 		(pts
+			(xy 226.06 416.56) (xy 226.06 417.83)
+		)
+		(stroke
+			(width 0)
+			(type default)
+		)
+	)
+	(wire
+		(pts
 			(xy 480.06 378.46) (xy 501.65 378.46)
 		)
@@
 		(dnp no)
 		(fields_autoplaced yes)
-		(property "Reference" "TP13"
+		(property "Reference" "TP14"
 			(at 765.81 418.3379 0)
 			(effects
@@
 			(project "KNEE CONTROLLER PCBA"
 				(path "/f9e05184-c88b-4a88-ae9c-ab2bdb32be7c/c5103ceb-5325-4a84-a025-9638a412984e"
-					(reference "TP13")
+					(reference "TP14")
 					(unit 1)
 				)
@@
 	)
 	(symbol
+		(lib_id "Connector:TestPoint")
+		(at 255.27 415.29 0)
+		(unit 1)
+		(exclude_from_sim no)
+		(in_bom no)
+		(on_board yes)
+		(dnp no)
+		(property "Reference" "TP13"
+			(at 255.27 406.4 0)
+			(effects
+				(font
+					(size 1.27 1.27)
+				)
+			)
+		)
+		(property "Value" "GND"
+			(at 255.27 408.94 0)
+			(effects
+				(font
+					(size 1.27 1.27)
+				)
+			)
+		)
+		(property "Footprint" "RD-Testpoints:TestPoint_Pad_1.0x1.0mm"
+			(at 260.35 415.29 0)
+			(effects
+				(font
+					(size 1.27 1.27)
+				)
+				(hide yes)
+			)
+		)
+		(property "Datasheet" "~"
+			(at 260.35 415.29 0)
+			(effects
+				(font
+					(size 1.27 1.27)
+				)
+				(hide yes)
+			)
+		)
+		(property "Description" "test point"
+			(at 255.27 415.29 0)
+			(effects
+				(font
+					(size 1.27 1.27)
+				)
+				(hide yes)
+			)
+		)
+		(property "Config" ""
+			(at 255.27 415.29 90)
+			(effects
+				(font
+					(size 1.27 1.27)
+				)
+				(hide yes)
+			)
+		)
+		(property "Sim.Device" ""
+			(at 255.27 415.29 0)
+			(effects
+				(font
+					(size 1.27 1.27)
+				)
+				(hide yes)
+			)
+		)
+		(property "Sim.Pins" ""
+			(at 255.27 415.29 0)
+			(effects
+				(font
+					(size 1.27 1.27)
+				)
+				(hide yes)
+			)
+		)
+		(property "Sim.Type" ""
+			(at 255.27 415.29 0)
+			(effects
+				(font
+					(size 1.27 1.27)
+				)
+				(hide yes)
+			)
+		)
+		(property "P_max" ""
+			(at 255.27 415.29 0)
+			(effects
+				(font
+					(size 1.27 1.27)
+				)
+				(hide yes)
+			)
+		)
+		(property "V_max" ""
+			(at 255.27 415.29 0)
+			(effects
+				(font
+					(size 1.27 1.27)
+				)
+				(hide yes)
+			)
+		)
+		(pin "1"
+		)
+		(instances
+			(project "KNEE CONTROLLER PCBA"
+				(path "/f9e05184-c88b-4a88-ae9c-ab2bdb32be7c/c5103ceb-5325-4a84-a025-9638a412984e"
+					(reference "TP13")
+					(unit 1)
+				)
+			)
+		)
+	)
+	(symbol
 		(lib_id "power:+BATT")
 		(at 73.66 152.4 0)
@@
 	(symbol
 		(lib_id "power:PWR_FLAG")
-		(at 255.27 415.29 0)
+		(at 226.06 417.83 180)
 		(unit 1)
 		(exclude_from_sim no)
@@
 		(fields_autoplaced yes)
 		(property "Reference" "#FLG011"
-			(at 255.27 413.385 0)
+			(at 226.06 419.735 0)
 			(effects
 				(font
@@
 		)
 		(property "Value" "PWR_FLAG"
-			(at 255.2699 411.48 90)
+			(at 226.0601 421.64 90)
 			(effects
 				(font
@@
 		)
 		(property "Footprint" ""
-			(at 255.27 415.29 0)
+			(at 226.06 417.83 0)
 			(effects
 				(font
@@
 		)
 		(property "Datasheet" "~"
-			(at 255.27 415.29 0)
+			(at 226.06 417.83 0)
 			(effects
 				(font
@@
 		)
 		(property "Description" "Special symbol for telling ERC where power comes from"
-			(at 255.27 415.29 0)
+			(at 226.06 417.83 0)
 			(effects
 				(font
