File: microcontroller.kicad_sch (KiCad schematic)
At the start: 65 parts, among them J2 USB_CONN, J3 ST-LINK_CONN, J4 TAG_CONN, SW1 SW_CAN_TERM, SW2 SW_USER, SW3 SW_RESET, U6 TJA1051T/3, U7 USBLC6-2SC6, U8 STM32L476RGT6, Y1 X50328MSB2GI, Y2 Q13FC13500004

Commit message: chore(pcb): update project files
Parts:
- added TP12: CAN_H, RD-Testpoints:TestPoint_Pad_D0.4mm, symbol Connector:TestPoint
- added TP13: CAN_L, RD-Testpoints:TestPoint_Pad_D0.4mm, symbol Connector:TestPoint
- added TP15: I2C2_SDA, RD-Testpoints:TestPoint_Pad_D0.4mm, symbol Connector:TestPoint
- added TP16: I2C2_SCL, RD-Testpoints:TestPoint_Pad_D0.4mm, symbol Connector:TestPoint
- added TP17: I2C1_SDA, RD-Testpoints:TestPoint_Pad_D0.4mm, symbol Connector:TestPoint
- added TP18: I2C1_SCL, RD-Testpoints:TestPoint_Pad_D0.4mm, symbol Connector:TestPoint
- renumbered TP9 to TP14
Connections:
- net CAN_H: now also TP12.1
- net CAN_L: now also TP13.1
- net I2C1_SCL: now also TP18.1
- net I2C1_SDA: now also TP17.1
- net I2C2_SCL: now also TP16.1
- net I2C2_SDA: now also TP15.1

Commit message: docs(docs): update project files
Parts:
- added TP19: CAN_RX, 0_RD_Testpoint:TestPoint_Pad_D0.4mm, symbol Connector:TestPoint
- added TP20: CAN _TX, 0_RD_Testpoint:TestPoint_Pad_D0.4mm, symbol Connector:TestPoint
- added TP21: CAN_S, 0_RD_Testpoint:TestPoint_Pad_D0.4mm, symbol Connector:TestPoint
- added TP26: DBG_RST_N, 0_RD_Testpoint:TestPoint_Pad_D0.4mm, symbol Connector:TestPoint
- C18, C36, C37: footprint Capacitor_SMD:C_0805_2012Metric -> 0_RD_Capacitor_SMD:C_0805_2012_DensityHigh
- C19, C20, C21, C22, C23, C24, C25, C29, C30, C31, C32, C33, C34, C35: footprint Capacitor_SMD:C_0603_1608Metric -> 0_RD_Capacitor_SMD:C_0603_1608_DensityHigh
- C26, C27: footprint Capacitor_SMD:C_0402_1005Metric -> 0_RD_Capacitor_SMD:C_0402_1005_DensityHigh
- C28: footprint Capacitor_SMD:C_1206_3216Metric -> 0_RD_Capacitor_SMD:C_1206_3216_DensityHigh
- D5: value TVS -> SMBJ5.0A-TR; footprint Diode_SMD:D_SMB -> 0_RD_Diode_SMD:D_SMB; I_peak (none) -> 68A; MPN (none) -> SMBJ5.0A-TR; Manufacturer (none) -> STMicroelectronics; SPN (none) -> 497-3144-1-ND; Supplier (none) -> DigiKey; now fitted; now in the parts list
- D6, D7: footprint LED_SMD:LED_0805_2012Metric -> 0_RD_LED_SMD:LED_0805_2012_DensityHigh
- FB1: footprint Inductor_SMD:L_0603_1608Metric -> 0_RD_Resistor_SMD:R_0603_1608_DensityHigh
- J4: footprint Connector:Tag-Connect_TC2030-IDC-NL_2x03_P1.27mm_Vertical -> 0_RD_Testpoint:Tag-Connect_TC2030-IDC-NL_2x03_P1.27mm_Vertical
- R23, R24, R25, R26, R27, R28, R29, R30, R31, R33, R34, R35, R36, R37, R39, R40, R41, R42, R43, R44, R45, R46, R47: footprint Resistor_SMD:R_0603_1608Metric -> 0_RD_Resistor_SMD:R_0603_1608_DensityHigh
- R32: footprint Resistor_SMD:R_0603_1608Metric -> 0_RD_Resistor_SMD:R_0603_1608_DensityLow
- R38: footprint Resistor_SMD:R_0402_1005Metric -> 0_RD_Resistor_SMD:R_0402_1005_DensityHigh
- SW2, SW3: footprint PTS526SxxxSMTR2:SW_SPST_PTS526xxxSMTR -> 0_Switch_SMD:SW_SPST_PTS526xxxSMTR
- TP16: renamed from TP12; footprint RD-Testpoints:TestPoint_Pad_D0.4mm -> 0_RD_Testpoint:TestPoint_Pad_D0.4mm
- TP17: renamed from TP13; footprint RD-Testpoints:TestPoint_Pad_D0.4mm -> 0_RD_Testpoint:TestPoint_Pad_D0.4mm
- TP18: renamed from TP14; footprint RD-Testpoints:TestPoint_Pad_D1.0mm -> 0_RD_Testpoint:TestPoint_Pad_D1.0mm
- TP22: renamed from TP15; footprint RD-Testpoints:TestPoint_Pad_D0.4mm -> 0_RD_Testpoint:TestPoint_Pad_D0.4mm
- TP23: renamed from TP16; footprint RD-Testpoints:TestPoint_Pad_D0.4mm -> 0_RD_Testpoint:TestPoint_Pad_D0.4mm
- TP24: renamed from TP17; footprint RD-Testpoints:TestPoint_Pad_D0.4mm -> 0_RD_Testpoint:TestPoint_Pad_D0.4mm
- TP25: renamed from TP18; footprint RD-Testpoints:TestPoint_Pad_D0.4mm -> 0_RD_Testpoint:TestPoint_Pad_D0.4mm
Connections:
- net +3V3: no longer FB1.2
- net CAN_RX: now also TP19.1
- net CAN_S: now also TP21.1
- net CAN_TX: now also TP20.1
- net DBG_RST_N: now also TP26.1
- net VDD: now also FB1.2
Other:
- moved on the sheet: C19
