File: motor-control.kicad_sch (KiCad schematic)
At the start: 13 parts, among them J3 MOT_CONN, J4 DRV_DIAG, J5 DRV_SKT_LEFT, J6 DRV_SKT_RIGHT, U5 TMC5160T Pro

Commit message: chore(pcb): update project files
Parts:
- removed C24: 100n, Capacitor_SMD:C_0603_1608Metric, symbol Device:C
- removed JP3: DRV_JMP_UART, Connector_PinHeader_2.54mm:PinHeader_1x02_P2.54mm_Vertical, symbol Jumper:Jumper_2_Open
- removed JP4: DRV_JMP_SPI, Connector_PinHeader_2.54mm:PinHeader_2x04_P2.54mm_Vertical, symbol Connector_Generic:Conn_02x04_Odd_Even
- added C38, C43, C44, C45, C46: 100n, Capacitor_SMD:C_0603_1608Metric, symbol Device:C
- added C39: 1u, Capacitor_SMD:C_1206_3216Metric, symbol Device:C
- added C41: 1u, Capacitor_SMD:C_0805_2012Metric, symbol Device:C
- added C42: 10n, Capacitor_SMD:C_0603_1608Metric, symbol Device:C
- added FID1, FID2, FID3: FIDUCIAL, Fiducial:Fiducial_1mm_Mask2mm, symbol Mechanical:Fiducial
- added H1, H2, H3, H4: MOUNT_M2.5, MountingHole:MountingHole_2.7mm_M2.5_ISO7380_Pad, symbol Mechanical:MountingHole_Pad
- added ID1: BOARD_STACKUP_MARKER, RD-Symbols-Silkscreen:STACKUP_ID_2L, symbol Ryan-Dynamics:BOARD_STACKUP_MARKER
- added ID2: BOARD_IDENTIFICATION_MARKER, RD-Symbols-Silkscreen:BOARD_IDENTIFICATION, symbol Ryan-Dynamics:BOARD_IDENTIFICATION_MARKER
- added J10: ADC_CONN, Connector_Molex:Molex_KK-254_AE-6410-03A_1x03_P2.54mm_Vertical, symbol Connector:Conn_01x03_Pin
- added J11: ENC_CONN, Connector_Molex:Molex_KK-254_AE-6410-06A_1x06_P2.54mm_Vertical, symbol Connector:Conn_01x06_Pin
- added J12: UART_CONN, Connector_Molex:Molex_KK-254_AE-6410-04A_1x04_P2.54mm_Vertical, symbol Connector:Conn_01x04_Pin
- added J13: CAN_CONN, Connector_Molex:Molex_KK-254_AE-6410-03A_1x03_P2.54mm_Vertical, symbol Connector:Conn_01x03_Pin
- added J14: I2C_CONN, Connector_Molex:Molex_KK-254_AE-6410-04A_1x04_P2.54mm_Vertical, symbol Connector:Conn_01x04_Pin
- added J15: SW1_CONN, Connector_PinHeader_2.54mm:PinHeader_1x03_P2.54mm_Vertical, symbol Connector:Conn_01x03_Pin
- added J16: SW2_CONN, Connector_PinHeader_2.54mm:PinHeader_1x03_P2.54mm_Vertical, symbol Connector:Conn_01x03_Pin
- added J17: SW3_CONN, Connector_PinHeader_2.54mm:PinHeader_1x03_P2.54mm_Vertical, symbol Connector:Conn_01x03_Pin
- added J18: SW4_CONN, Connector_PinHeader_2.54mm:PinHeader_1x03_P2.54mm_Vertical, symbol Connector:Conn_01x03_Pin
- added J5: TEMP_CONN, Connector_Molex:Molex_KK-254_AE-6410-02A_1x02_P2.54mm_Vertical, symbol Connector:Conn_01x02_Pin
- added R50: 47k, Resistor_SMD:R_0603_1608Metric, symbol Device:R
- added R51: 100, Resistor_SMD:R_0603_1608Metric, symbol Device:R
- added R52: 1k, Resistor_SMD:R_0603_1608Metric, symbol Device:R
- added R53, R54, R55, R56: 10k, Resistor_SMD:R_0603_1608Metric, symbol Device:R
- added TH1: NTC100k, symbol Device:Thermistor_NTC
- added TP10, TP11, TP12: GND, RD-Testpoints:TestPoint_Pad_1.0x1.0mm, symbol Connector:TestPoint
- added TP13: TEMP_ADC, RD-Testpoints:TestPoint_Pad_D0.4mm, symbol Connector:TestPoint
- added TP14: AUX_ADC, RD-Testpoints:TestPoint_Pad_D0.4mm, symbol Connector:TestPoint
- C40: renamed from C23; footprint (none) -> Capacitor_THT:CP_Radial_D8.0mm_P3.50mm; Dielectric (none) -> Aluminium Electrolytic; Lifetime (none) -> 1000 Hrs @ 105°C; MPN C1608X7R0J106KT -> 63PX100MEFC8X11.5; Manufacturer TPK -> Rubycon; SPN (none) -> 1189-63PX100MEFC8X11.5-ND; SPN2 (none) -> C88774; Supplier (none) -> DigiKey; Supplier2 (none) -> LCSC; Tolerance 10% -> 20%; Voltage_Rating 100V -> 63V
- J6: renamed from J4; MPN (none) -> HX PM2.54-1x2P ZC H11; Manufacturer (none) -> hanxia; SPN (none) -> C41427517; Supplier (none) -> LCSC
- J7: renamed from J5; MPN (none) -> HX PM2.54-1x8P ZC H11; Manufacturer (none) -> hanxia; SPN (none) -> C41427523; Supplier (none) -> LCSC
- J8: renamed from J6; MPN (none) -> HX PM2.54-1x8P ZC H11; Manufacturer (none) -> hanxia; SPN (none) -> C41427523; Supplier (none) -> LCSC
- J9: renamed from J3; footprint (none) -> Connector_Molex_Addendum:Molex_Micro-Fit_3.0_43650-0415_1x04_P3.00mm_Vertical; symbol Connector:Conn_01x04_Socket -> Connector:Conn_01x04_Pin; MPN (none) -> 0436500415; MPN2 (none) -> C3030WV-4P; Manufacturer (none) -> Molex; Manufacturer2 (none) -> CJT(Changjiang Connectors); SPN (none) -> WM1919-ND; SPN2 (none) -> C239441; Supplier (none) -> DigiKey; Supplier2 (none) -> LCSC
- JP3: renamed from JP2; footprint Connector_PinHeader_2.54mm:PinHeader_1x04_P2.54mm_Vertical -> Jumpers:PinHeader_1x04_P2.54mm_Vertical; symbol Connector:Conn_01x04_Pin -> Jumpers:Conn_01x04_Pin; MPN (none) -> HM3212; MPN2 (none) -> HX PZ2.54-1x4P ZZ; Manufacturer (none) -> Jaycar Electronics; Manufacturer2 (none) -> hanxia; SPN (none) -> HM3212; SPN2 (none) -> C32713270; Supplier (none) -> Jaycar Electronics; Supplier2 (none) -> LCSC
- JP4: renamed from JP1; footprint Connector_PinHeader_2.54mm:PinHeader_2x04_P2.54mm_Vertical -> Jumpers:PinHeader_2x04_P2.54mm_Vertical; MPN (none) -> HM3250; MPN2 (none) -> HX PZ2.54-2x4P ZZ; Manufacturer (none) -> Jaycar Electronics; Manufacturer2 (none) -> hanxia; SPN (none) -> HM3250; SPN2 (none) -> C32713277; Supplier (none) -> Jaycar Electronics; Supplier2 (none) -> LCSC
- R48: renamed from R10; MPN (none) -> RT0603FRE071KL; MPN2 (none) -> 0603WAF1001T5E; Manufacturer (none) -> YAGEO; Manufacturer2 (none) -> UNI-ROYAL; Power_Rating (none) -> 1/10W; SPN (none) -> YAG2323CT-ND; SPN2 (none) -> C21190; Supplier (none) -> DigiKey; Supplier2 (none) -> LCSC; Tolerance (none) -> 1%; Voltage_Rating (none) -> 75V
- R49: renamed from R11; MPN (none) -> RT0603FRE1010KL; MPN2 (none) -> 0603WAF1002T5E; Manufacturer (none) -> YAGEO; Manufacturer2 (none) -> UNI-ROYAL; Power_Rating (none) -> 1/10W; SPN (none) -> 13-RT0603FRE1010KLCT-ND; SPN2 (none) -> C25804; Supplier (none) -> DigiKey; Supplier2 (none) -> LCSC; Tolerance (none) -> 1%; Voltage_Rating (none) -> 75V
- U9: renamed from U5; Cost (none) -> $34.45; SPN TMC5160T Pro -> 1050000063; Supplier BIGTREETECH -> DREMC
Connections:
- net +3V3: now also J10.2 (Pin_2), J11.2 (Pin_2), J12.2 (Pin_2), J14.2 (Pin_2), J15.2 (Pin_2), J16.2 (Pin_2), J17.2 (Pin_2), J18.2 (Pin_2), R50.2, R53.1, R54.1, R55.1, R56.1
- net B1: now also J8.6 (Pin_6), J9.1 (Pin_1), U9.11 (B1); no longer J8.5 (Pin_5), J9.2 (Pin_2), U9.12 (B1)
- net B2: now also J8.5 (Pin_5), J9.2 (Pin_2), U9.12 (B2); no longer J8.6 (Pin_6), J9.1 (Pin_1), U9.11 (B2)
- net GND: now also C38.2, C39.1, C41.1, C42.1, C43.1, C44.1, C45.1, C46.1, H1.1, H2.1, H3.1, H4.1, J10.1 (Pin_1), J11.1 (Pin_1), J12.1 (Pin_1), J13.1 (Pin_1), J14.1 (Pin_1), J15.1 (Pin_1), J16.1 (Pin_1), J17.1 (Pin_1), J18.1 (Pin_1), J5.1 (Pin_1), TH1.2, TP10.1, TP11.1, TP12.1
- net +BATT renamed +VM
- net +VM: now also C38.1, C39.2
- net DRV_CSN renamed DRV_CS
- net DRV_SDI renamed DRV_MOSI
- net DRV_SDO renamed DRV_MISO
- net DRV_~{EN} renamed DRV_EN_N
- new net AUX_ADC: C42.2, R52.2, TP14.1
- new net AUX_ADC_CONN: J10.3 (Pin_3), R52.1
- new net AUX_UART_RX: J12.4 (Pin_4)
- new net AUX_UART_TX: J12.3 (Pin_3)
- new net CAN_H: J13.3 (Pin_3)
- new net CAN_L: J13.2 (Pin_2)
- new net ENC_AUX_SCK: J11.3 (Pin_3)
- new net ENC_A_MISO: J11.4 (Pin_4)
- new net ENC_B_MOSI: J11.5 (Pin_5)
- new net ENC_Z_CS: J11.6 (Pin_6)
- new net I2C2_SCL: J14.4 (Pin_4)
- new net I2C2_SDA: J14.3 (Pin_3)
- new net SW1_SIG: C43.2, J15.3 (Pin_3), R53.2
- new net SW2_SIG: C44.2, J16.3 (Pin_3), R54.2
- new net SW3_SIG: C45.2, J17.3 (Pin_3), R55.2
- new net SW4_SIG: C46.2, J18.3 (Pin_3), R56.2
- new net TEMP_ADC: C41.2, R51.2, TP13.1
- new net TEMP_NTC: J5.2 (Pin_2), R50.1, R51.1, TH1.1
Other:
- note added: "MARKINGS"
- note added: "MOUNTING"
- note added: "SPEED STICK SOCKET"
- note removed: "SPI/UART JUMPERS"
- title: DIGITAL -> MOTOR CONTROL AND IO
- moved on the sheet: C40, J6, J7, J8, JP3, JP4, R48, R49, U9

Commit message: chore(pcb): update project files
Parts:
- added TP24: GND, RD-Testpoints:TestPoint_Pad_1.0x1.0mm, symbol Connector:TestPoint
- renumbered TP10 to TP19, TP11 to TP20, TP12 to TP21, TP13 to TP22, TP14 to TP23
Connections:
- net GND: now also TP24.1
Other:
- moved on the sheet: H1, H2, H3, H4, TP19, TP20, TP21

Commit message: docs(docs): update project files
Parts:
- added TP31: DRV_MISO, 0_RD_Testpoint:TestPoint_Pad_D0.4mm, symbol Connector:TestPoint
- added TP32: DRV_MOSI, 0_RD_Testpoint:TestPoint_Pad_D0.4mm, symbol Connector:TestPoint
- added TP33: DRV_SCK, 0_RD_Testpoint:TestPoint_Pad_D0.4mm, symbol Connector:TestPoint
- added TP34: DRV_CS, 0_RD_Testpoint:TestPoint_Pad_D0.4mm, symbol Connector:TestPoint
- added TP35: DRV_DIR, 0_RD_Testpoint:TestPoint_Pad_D0.4mm, symbol Connector:TestPoint
- added TP36: DRV_EN_N, 0_RD_Testpoint:TestPoint_Pad_D0.4mm, symbol Connector:TestPoint
- added TP37: STEP_DIR, 0_RD_Testpoint:TestPoint_Pad_D0.4mm, symbol Connector:TestPoint
- added TP39: ENC_AUX_SCK, 0_RD_Testpoint:TestPoint_Pad_D0.4mm, symbol Connector:TestPoint
- added TP40: ENC_A_MISO, 0_RD_Testpoint:TestPoint_Pad_D0.4mm, symbol Connector:TestPoint
- added TP41: ENC_B_MOSI, 0_RD_Testpoint:TestPoint_Pad_D0.4mm, symbol Connector:TestPoint
- added TP42: ENC_Z_CS, 0_RD_Testpoint:TestPoint_Pad_D0.4mm, symbol Connector:TestPoint
- C38, C42, C43, C44, C45, C46: footprint Capacitor_SMD:C_0603_1608Metric -> 0_RD_Capacitor_SMD:C_0603_1608_DensityHigh
- C39: footprint Capacitor_SMD:C_1206_3216Metric -> 0_RD_Capacitor_SMD:C_1206_3216_DensityHigh
- C41: footprint Capacitor_SMD:C_0805_2012Metric -> 0_RD_Capacitor_SMD:C_0805_2012_DensityHigh
- FID1, FID2, FID3: footprint Fiducial:Fiducial_1mm_Mask2mm -> 0_RD_Fiducial:Fiducial_1mm_Mask2mm
- ID1: footprint RD-Symbols-Silkscreen:STACKUP_ID_2L -> 0_RD_Identification:STACKUP_ID_2L
- ID2: footprint RD-Symbols-Silkscreen:BOARD_IDENTIFICATION -> 0_RD_Identification:BOARD_IDENTIFICATION
- J9: footprint Connector_Molex_Addendum:Molex_Micro-Fit_3.0_43650-0415_1x04_P3.00mm_Vertical -> 0_Connector:Molex_Micro-Fit_3.0_43650-0415_1x04_P3.00mm_Vertical
- JP3: footprint Jumpers:PinHeader_1x04_P2.54mm_Vertical -> 0_Jumper:PinHeader_1x04_P2.54mm_Vertical
- JP4: footprint Jumpers:PinHeader_2x04_P2.54mm_Vertical -> 0_Jumper:PinHeader_2x04_P2.54mm_Vertical
- R48, R49, R50, R51, R52, R53, R54, R55, R56: footprint Resistor_SMD:R_0603_1608Metric -> 0_RD_Resistor_SMD:R_0603_1608_DensityHigh
- TP27: renamed from TP19; value GND -> G; footprint RD-Testpoints:TestPoint_Pad_1.0x1.0mm -> 0_RD_Testpoint:TestPoint_Pad_1.0x1.0mm
- TP28: renamed from TP24; value GND -> G; footprint RD-Testpoints:TestPoint_Pad_1.0x1.0mm -> 0_RD_Testpoint:TestPoint_Pad_1.0x1.0mm
- TP29: renamed from TP20; value GND -> G; footprint RD-Testpoints:TestPoint_Pad_1.0x1.0mm -> 0_RD_Testpoint:TestPoint_Pad_1.0x1.0mm
- TP30: renamed from TP21; value GND -> G; footprint RD-Testpoints:TestPoint_Pad_1.0x1.0mm -> 0_RD_Testpoint:TestPoint_Pad_1.0x1.0mm
- TP38: renamed from TP22; footprint RD-Testpoints:TestPoint_Pad_D0.4mm -> 0_RD_Testpoint:TestPoint_Pad_D0.4mm
- TP43: renamed from TP23; footprint RD-Testpoints:TestPoint_Pad_D0.4mm -> 0_RD_Testpoint:TestPoint_Pad_D0.4mm
- U9: footprint (none) -> 0_Module:TMC5160T PRO
Connections:
- net DRV_CS: now also TP34.1
- net DRV_DIR: now also TP35.1
- net DRV_EN_N: now also TP36.1
- net DRV_MISO: now also TP31.1
- net DRV_MOSI: now also TP32.1
- net DRV_SCK: now also TP33.1
- net DRV_STEP: now also TP37.1
- net ENC_AUX_SCK: now also TP39.1
- net ENC_A_MISO: now also TP40.1
- net ENC_B_MOSI: now also TP41.1
- net ENC_Z_CS: now also TP42.1
Other:
- moved on the sheet: JP3, JP4, R48
