File: power-management.kicad_sch (KiCad schematic)
At the start: 61 parts, among them J1 VIN_CONN, Q1 CRTD700P10L, Q2 NCE0106R, U1 INA238AIDGSR, U2 TLV4041R5DBVR, U3 TLV6700QDDCRQ1, U4 LMR36510ADDAR, U5 AP7362-33SP-13

Commit message: chore(pcb): update project files
Parts:
- added TP7: SW, RD-Testpoints:TestPoint_Pad_D0.4mm, symbol Connector:TestPoint
- added TP8: VIN_SEL, RD-Testpoints:TestPoint_Pad_D0.4mm, symbol Connector:TestPoint
- added TP9: FB, RD-Testpoints:TestPoint_Pad_D0.4mm, symbol Connector:TestPoint
- renumbered TP7 to TP10, TP8 to TP11
Connections:
- net FB: now also TP9.1
- net SW: now also TP7.1
- net VIN_SEL: now also TP8.1

Commit message: docs(docs): update project files
Parts:
- added TP2: BRAKE_SENSE, 0_RD_Testpoint:TestPoint_Pad_D0.4mm, symbol Connector:TestPoint
- added TP4: RPP_GATE, 0_RD_Testpoint:TestPoint_Pad_D0.4mm, symbol Connector:TestPoint
- added TP5: BRAKE_CMD, 0_RD_Testpoint:TestPoint_Pad_D0.4mm, symbol Connector:TestPoint
- added TP6: BRAKE_GATE, 0_RD_Testpoint:TestPoint_Pad_D0.4mm, symbol Connector:TestPoint
- C1, C12, C16, C2, C4, C5, C6, C7: footprint Capacitor_SMD:C_0603_1608Metric -> 0_RD_Capacitor_SMD:C_0603_1608_DensityHigh
- C10, C11, C15, C17: footprint Capacitor_SMD:C_0805_2012Metric -> 0_RD_Capacitor_SMD:C_0805_2012_DensityHigh
- C13, C14, C8, C9: footprint Capacitor_SMD:C_1206_3216Metric -> 0_RD_Capacitor_SMD:C_1206_3216_DensityHigh
- D1: footprint Diode_SMD:D_SOD-323_HandSoldering -> 0_RD_Diode_SMD:D_SOD-323
- D2, D3: footprint LED_SMD:LED_0805_2012Metric -> 0_RD_LED_SMD:LED_0805_2012_DensityHigh
- J1: footprint Connector_Molex_Addendum:Molex_Micro-Fit_3.0_43650-0215_1x02_P3.00mm_Vertical -> 0_Connector:Molex_KK-396_5273-02A_1x02_P3.96mm_Vertical
- R1, R10, R11, R13, R16, R17, R18, R19, R2, R20, R21, R22, R3, R4, R5, R6, R7, R8, R9: footprint Resistor_SMD:R_0603_1608Metric -> 0_RD_Resistor_SMD:R_0603_1608_DensityHigh
- TP1: footprint RD-Testpoints:TestPoint_Pad_D1.0mm -> 0_RD_Testpoint:TestPoint_Pad_D1.0mm
- TP10: renamed from TP6; footprint RD-Testpoints:TestPoint_Pad_D0.4mm -> 0_RD_Testpoint:TestPoint_Pad_D0.4mm
- TP11: renamed from TP7; footprint RD-Testpoints:TestPoint_Pad_D0.4mm -> 0_RD_Testpoint:TestPoint_Pad_D0.4mm
- TP12: renamed from TP8; footprint RD-Testpoints:TestPoint_Pad_D0.4mm -> 0_RD_Testpoint:TestPoint_Pad_D0.4mm
- TP13: renamed from TP9; footprint RD-Testpoints:TestPoint_Pad_D0.4mm -> 0_RD_Testpoint:TestPoint_Pad_D0.4mm
- TP14: renamed from TP10; footprint RD-Testpoints:TestPoint_Pad_D1.0mm -> 0_RD_Testpoint:TestPoint_Pad_D1.0mm
- TP15: renamed from TP11; footprint RD-Testpoints:TestPoint_Pad_D1.0mm -> 0_RD_Testpoint:TestPoint_Pad_D1.0mm
- TP3: renamed from TP2; footprint RD-Testpoints:TestPoint_Pad_D0.4mm -> 0_RD_Testpoint:TestPoint_Pad_D0.4mm
- TP7: renamed from TP3; footprint RD-Testpoints:TestPoint_Pad_D1.0mm -> 0_RD_Testpoint:TestPoint_Pad_D1.0mm
- TP8: renamed from TP4; footprint RD-Testpoints:TestPoint_Pad_D1.0mm -> 0_RD_Testpoint:TestPoint_Pad_D1.0mm
- TP9: renamed from TP5; footprint RD-Testpoints:TestPoint_Pad_D0.4mm -> 0_RD_Testpoint:TestPoint_Pad_D0.4mm
- U5: footprint AP7362-33SP-13:SOIC-8-1EP_3.9x4.9mm_P1.27mm_EP2.6x3.5mm_ThermalVias -> 0_SOIC:SOIC-8-1EP_3.9x4.9mm_P1.27mm_EP2.6x3.5mm_ThermalVias
Connections:
- net BRAKE_CMD: now also TP5.1
- net BRAKE_GATE: now also TP6.1
- net BRAKE_SENSE: now also TP2.1
- net RPP_GATE: now also TP4.1
Other:
- moved on the sheet: R1

Commit message: chore(pcb): update project files
Changed lines of the file:
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@@
 		)
 	)
-	(text_box "DESIGN NOTE:\nFH1 = MINI BLADE FUSE HOLDER\nUSE 58 VDC-RATED FUSE\nFUSE CURRENT RATING TBD"
+	(text_box "DESIGN NOTE:\nFH1 = MINI BLADE FUSE HOLDER\nUSE 58 VDC-RATED FUSE\nFUSE CURRENT RATING 5A"
 		(exclude_from_sim no)
 		(at 85.09 39.37 0)
-		(size 27.94 13.97)
+		(size 27.94 12.7)
 		(margins 1.3525 1.3525 1.3525 1.3525)
 		(stroke
