File: KNEE CONTROLLER PCBA.kicad_sch (KiCad schematic)
At the start: 0 parts

Commit message: chore(pcb): update project files
Other:
- removed sheet BLOCK DIAGRAM
- removed sheet POWER SEQUENCE
Changed lines of the file:
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@@
 		(exclude_from_sim no)
 		(at 123.19 166.37 0)
-		(size 69.85 78.74)
+		(size 44.45 53.34)
 		(margins 1.905 1.905 1.905 1.905)
 		(stroke
@@
 		(exclude_from_sim no)
 		(at 22.86 166.37 0)
-		(size 69.85 78.74)
+		(size 46.99 53.34)
 		(margins 1.905 1.905 1.905 1.905)
 		(stroke
@@
 	)
 	(sheet
-		(at 340.36 313.69)
+		(at 340.36 302.26)
 		(size 35.56 5.08)
 		(exclude_from_sim no)
@@
 		(dnp no)
 		(stroke
-			(width 0.1524)
+			(width 0)
 			(type solid)
 		)
@@
 			(color 0 0 0 0.0000)
 		)
-		(property "Sheetname" "POWER SEQUENCE"
-			(at 340.36 312.6609 0)
+		(property "Sheetname" "REVISION HISTORY"
+			(at 340.36 300.99 0)
 			(effects
 				(font
@@
 			)
 		)
-		(property "Sheetfile" "power-sequence.kicad_sch"
-			(at 341.63 314.96 0)
+		(property "Sheetfile" "revision-history.kicad_sch"
+			(at 340.995 303.53 0)
 			(effects
 				(font
@@
 			(project "KNEE CONTROLLER PCBA"
 				(path "/f9e05184-c88b-4a88-ae9c-ab2bdb32be7c"
-					(page "6")
+					(page "3")
 				)
 			)
@@
 	)
 	(sheet
-		(at 340.36 302.26)
+		(at 299.72 313.69)
 		(size 35.56 5.08)
 		(exclude_from_sim no)
@@
 		(dnp no)
 		(stroke
-			(width 0)
+			(width 0.1524)
 			(type solid)
 		)
@@
 			(color 0 0 0 0.0000)
 		)
-		(property "Sheetname" "REVISION HISTORY"
-			(at 340.36 300.99 0)
+		(property "Sheetname" "PROJECT"
+			(at 299.72 312.6609 0)
 			(effects
 				(font
@@
 			)
 		)
-		(property "Sheetfile" "revision-history.kicad_sch"
-			(at 340.995 303.53 0)
-			(effects
-				(font
-					(face "Arimo")
-					(size 1.27 1.27)
-				)
-				(justify left top)
-			)
-		)
-		(instances
-			(project "KNEE CONTROLLER PCBA"
-				(path "/f9e05184-c88b-4a88-ae9c-ab2bdb32be7c"
-					(page "7")
-				)
-			)
-		)
-	)
-	(sheet
-		(at 299.72 302.26)
-		(size 35.56 5.08)
-		(exclude_from_sim no)
-		(in_bom yes)
-		(on_board yes)
-		(dnp no)
-		(stroke
-			(width 0.1524)
-			(type solid)
-		)
-		(fill
-			(color 0 0 0 0.0000)
-		)
-		(property "Sheetname" "BLOCK DIAGRAM"
-			(at 299.72 301.2309 0)
-			(effects
-				(font
-					(face "Tinos")
-					(size 1.905 1.905)
-					(bold yes)
-					(color 0 0 0 1)
-				)
-				(justify left bottom)
-			)
-		)
-		(property "Sheetfile" "block-diagram.kicad_sch"
-			(at 300.99 303.53 0)
+		(property "Sheetfile" "project.kicad_sch"
+			(at 300.99 314.96 0)
 			(effects
 				(font
@@
 				)
 			)
-		)
-	)
-	(sheet
-		(at 299.72 313.69)
-		(size 35.56 5.08)
-		(exclude_from_sim no)
-		(in_bom yes)
-		(on_board yes)
-		(dnp no)
-		(stroke
-			(width 0.1524)
-			(type solid)
-		)
-		(fill
-			(color 0 0 0 0.0000)
-		)
-		(property "Sheetname" "PROJECT"
-			(at 299.72 312.6609 0)
-			(effects
-				(font
-					(face "Tinos")
-					(size 1.905 1.905)
-					(bold yes)
-					(color 0 0 0 1)
-				)
-				(justify left bottom)
-			)
-		)
-		(property "Sheetfile" "project.kicad_sch"
-			(at 300.99 314.96 0)
-			(effects
-				(font
-					(face "Arimo")
-					(size 1.27 1.27)
-				)
-				(justify left top)
-			)
-		)
-		(instances
-			(project "KNEE CONTROLLER PCBA"
-				(path "/f9e05184-c88b-4a88-ae9c-ab2bdb32be7c"
-					(page "3")
-				)
-			)

Commit message: chore(pcb): update project files
Other:
- removed sheet PROJECT
- removed sheet REVISION HISTORY
- added sheet SYSTEM OVERVIEW (system-overview.kicad_sch)
- title: (none) -> COVER PAGE
Changed lines of the file:
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@@
 	(paper "A3")
 	(title_block
-		(date "2025-01-12")
+		(title "COVER PAGE")
+		(date "2026-10-12")
 		(rev "${DRAWING_REVISION}")
 		(company "${COMPANY}")
@@
 	)
 	(sheet
-		(at 340.36 302.26)
+		(at 299.72 326.39)
 		(size 35.56 5.08)
 		(exclude_from_sim no)
@@
 		(dnp no)
 		(stroke
-			(width 0)
+			(width 0.1524)
 			(type solid)
 		)
@@
 			(color 0 0 0 0.0000)
 		)
-		(property "Sheetname" "REVISION HISTORY"
-			(at 340.36 300.99 0)
+		(property "Sheetname" "SYSTEM OVERVIEW"
+			(at 299.72 325.3609 0)
 			(effects
 				(font
@@
 			)
 		)
-		(property "Sheetfile" "revision-history.kicad_sch"
-			(at 340.995 303.53 0)
+		(property "Sheetfile" "system-overview.kicad_sch"
+			(at 300.99 327.66 0)
 			(effects
 				(font
-					(face "Arimo")
-					(size 1.27 1.27)
-				)
-				(justify left top)
-			)
-		)
-		(instances
-			(project "KNEE CONTROLLER PCBA"
-				(path "/f9e05184-c88b-4a88-ae9c-ab2bdb32be7c"
-					(page "3")
-				)
-			)
-		)
-	)
-	(sheet
-		(at 299.72 313.69)
-		(size 35.56 5.08)
-		(exclude_from_sim no)
-		(in_bom yes)
-		(on_board yes)
-		(dnp no)
-		(stroke
-			(width 0.1524)
-			(type solid)
-		)
-		(fill
-			(color 0 0 0 0.0000)
-		)
-		(property "Sheetname" "PROJECT"
-			(at 299.72 312.6609 0)
-			(effects
-				(font
-					(face "Tinos")
-					(size 1.905 1.905)
-					(bold yes)
-					(color 0 0 0 1)
-				)
-				(justify left bottom)
-			)
-		)
-		(property "Sheetfile" "project.kicad_sch"
-			(at 300.99 314.96 0)
-			(effects
-				(font

Commit message: chore(pcb): update project files
Other:
- note added: "MADE WITH LOVE"
- note removed: "COMMENT"
